File: PCB/Gargamel/Gargamel-Amplifier.kicad_sch (KiCad schematic)
At the start: 14 parts, among them J1 8P8C_Shielded, U1 AD8608ARUZ-REEL

Commit message: save progress
Parts:
- U1: footprint RU_14_ADI -> AD8608ARUZ:RU_14_ADI
Changed lines of the file:
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@@
 			)
 		)
-		(property "Footprint" "RU_14_ADI"
+		(property "Footprint" "AD8608ARUZ:RU_14_ADI"
 			(at 139.7 77.47 0)
 			(effects
