File: PCB/Gargamel/Gargamel.kicad_sch (KiCad schematic)
At the start: 1 part, among them IC1 ADS131E08IPAGR

Commit message: finished SPI, working on ADC
Parts:
- added CS10, CS11, CS12, CS14, CS16, CS19, CS5, CS6, CS7, CS8, CS9: 1u, Capacitor_SMD:C_0603_1608Metric, symbol Device:C
- added CS13, CS20: 100n, Capacitor_SMD:C_0603_1608Metric, symbol Device:C
- added CS15: 22u, Capacitor_SMD:C_0603_1608Metric, symbol Device:C
- added CS17: 10u, Capacitor_SMD:C_0603_1608Metric, symbol Device:C
- added JP2: SolderJumper_2_Open, Jumper:SolderJumper-2_P1.3mm_Open_RoundedPad1.0x1.5mm, symbol Jumper:SolderJumper_2_Open
- added R4, R5, R6, R7, R8, R9: 10k, Resistor_SMD:R_0603_1608Metric, symbol Device:R
Connections:
- net 5V: now reaches IC1.19 (AVDD_1)
- net 5V: now also IC1.21 (AVDD_2), IC1.22 (AVDD_3), IC1.54 (AVDD1), IC1.56 (AVDD_4), IC1.59 (AVDD_5), CS10.2, CS5.2, CS6.2, CS7.2, CS8.2, CS9.2
- net GND: now reaches IC1.20 (AVSS_1)
- net GND: now also IC1.23 (AVSS_2), IC1.25 (VREFN), IC1.32 (AVSS_3), IC1.33 (DGND_1), IC1.37 (CLK), IC1.41 (DAISY_IN), IC1.49 (DGND_2), IC1.51 (DGND_3), IC1.53 (AVSS1), IC1.57 (AVSS_4), IC1.58 (AVSS_5), CS10.1, CS11.1, CS12.1, CS13.2, CS14.2, CS15.2, CS16.2, CS17.2, CS19.1, CS20.2, CS5.1, CS6.1, CS7.1, CS8.1, CS9.1, JP2.2 (B), R4.2, R5.2, R6.2, R7.2, R9.1
- net Ref_P: now reaches IC1.24 (VREFP)
- net Ref_P: now also CS17.1, CS20.1, R8.2
- net at IC1.26 (VCAP4): now also CS14.1
- net at IC1.28 (VCAP1): now also CS15.1
- net at IC1.30 (VCAP2): now also CS16.1
- net Output/MOSI: now reaches IC1.34 (DIN)
- net Output/CS*: now reaches IC1.39 (~{CS})
- net Output/SCK: now reaches IC1.40 (SCLK)
- net at IC1.42 (GPIO1): now also R7.1
- net at IC1.44 (GPIO2): now also R6.1
- net at IC1.45 (GPIO3): now also R5.1
- net at IC1.46 (GPIO4): now also R4.1
- net Output/SBU: now reaches IC1.47 (~{DRDY})
- net 3.3V: now reaches IC1.48 (DVDD_1)
- net 3.3V: now also IC1.50 (DVDD_2), IC1.52 (CLKSEL), CS11.2, CS19.2
- net at IC1.55 (VCAP3): now also CS12.2, CS13.1
- new net: R8.1, R9.2
- new net Shield: JP2.1 (A)
- no-connect marks 0 -> 4
Other:
- sheet Amlifier renamed Amplifier
- added sheet Output (Output.kicad_sch)
- note added: "1uF for each AVDD/DVDD input"
- note added: "Maybe LED for GPIO?"
- note added: "Programming: - Set SPI Mode (0,1) CPOL=0, CPHA=1 - Set internal Reference Voltage to 4V"
- note added: "active internal reference voltage"
- note added: "use internal opamp for bias + unity gain buffer"
- note removed: "LVDS: LTC6820 -> simple Pulse LTC4332 -> Dual Alternativ nach TIDA-060017: SN65LVDS31 DS90LV047A"
- note removed: "nochmal USB (!24pin wahrscheinlich): GT-USB-7045C 16pin: TYPE-C-31-M-12 -> D+/D-, SBU, CC, PWR+GND? alternativ nochmal rj45"
- moved on the sheet: IC1

Commit message: save progress
Parts:
- removed R8, R9: 10k, Resistor_SMD:R_0603_1608Metric, symbol Device:R
- added JP2: SolderJumper_3_Bridged12, symbol Jumper:SolderJumper_3_Bridged12
- added JP_ADC_RefP: SolderJumper_2_Open, Jumper:SolderJumper-2_P1.3mm_Open_RoundedPad1.0x1.5mm, symbol Jumper:SolderJumper_2_Open
- added TP_OPn, TP_OPout, TP_OPp: TestPoint, TestPoint:TestPoint_Pad_1.0x1.0mm, symbol Connector:TestPoint
- added TP_REFp: TestPoint, TestPoint:TestPoint_THTPad_D1.0mm_Drill0.5mm, symbol Connector:TestPoint
- renumbered JP2 to JP_Shield_GND
Connections:
- net 5V: now also JP_ADC_RefP.1 (A)
- net GND: now also IC1.1 (IN8N), IC1.11 (IN3N), IC1.13 (IN2N), IC1.15 (IN1N), IC1.3 (IN7N), IC1.5 (IN6N), IC1.7 (IN5N), IC1.9 (IN4N), JP2.3 (B)
- net Output/CC: now also JP2.1 (A)
- net Output/MISO: now also IC1.43 (DOUT)
- net at IC1.38 (START): now also JP2.2 (C)
- net at IC1.60 (OPAMPP): now also TP_OPp.1
- net at IC1.61 (OPAMPN): now also TP_OPn.1
- net at IC1.63 (OPAMPOUT): now also TP_OPout.1
- net Ref_P: no longer names the net of CS17.1, CS20.1, IC1.24 (VREFP)
- net Ref_P: now also JP_ADC_RefP.2 (B), TP_REFp.1
Other:
- added sheet Voltage Regulator (Regulator.kicad_sch)
- note added: "alternativley -> power down & supply external reference"
- note added: "use internal opamp + unity gain buffer for OP-Amp Bias"
- note removed: "use internal opamp for bias + unity gain buffer"
- moved on the sheet: CS10, CS11, CS19, CS5, CS6, CS7, CS8, CS9
