File: PCB/Schlaubi-Schlumpf/ADC.kicad_sch (KiCad schematic)
At the start: 42 parts, among them IC1 ADS131E08IPAGR, J1 8P8C_Shielded, J2 Conn_01x02_Pin, J3 Conn_01x02_Pin

Commit message: added IMU
Parts:
- renumbered TP_OPn1 to TP_OP_N, TP_OPout1 to TP_OP_OUT, TP_OPp1 to TP_OP_P
Connections:
- net *CS renamed ADC.*CS
- net *DRDY renamed ADC.*DRDY
- net MISO renamed ADC.MISO
- net MOSI renamed ADC.MOSI
- net SCLK renamed ADC.SCLK
- net START renamed ADC.START
Other:
- sheet Amplifier renamed Charge-Amplifier-Sensitive
- added sheet Charge-Amplifier-Coarse (Charge-Amplifier.kicad_sch)
- sheet Charge-Amplifier-Sensitive: file Gargamel-Amplifier.kicad_sch -> Charge-Amplifier.kicad_sch

Commit message: v1
Parts:
- removed CS15, CS32, CS33, CS34, CS35, CS36: 100n, Capacitor_SMD:C_0603_1608Metric, symbol Device:C
- removed CS31: 1u, Capacitor_SMD:C_0603_1608Metric, symbol Device:C
- removed J1: 8P8C_Shielded, symbol Connector:8P8C_Shielded
- added R18, R21, R22, R23, R24, R25, R26: 0R, Resistor_SMD:R_0603_1608Metric, symbol Device:R
- added R5: 100R, Resistor_SMD:R_0603_1608Metric, symbol Device:R
- added TP_GND1: TestPoint, TestPoint:TestPoint_Pad_D1.0mm, symbol Connector:TestPoint
- ADC_Daisy1: renamed from ADC_Daisy; footprint (none) -> TestPoint:TestPoint_Pad_D1.0mm
- ADC_TESTN1: renamed from ADC_TESTN; footprint (none) -> TestPoint:TestPoint_Pad_D1.0mm
- ADC_TESTP1: renamed from ADC_TESTP; footprint (none) -> TestPoint:TestPoint_Pad_D1.0mm
- CS11, CS9: value 1u -> 10u
- D3, D4: footprint (none) -> LED_SMD:LED_0603_1608Metric
- J2, J3: footprint (none) -> Connector_PinHeader_1.00mm:PinHeader_1x02_P1.00mm_Vertical
- R14: value 100R -> 0R
- TP_OP_N1: renamed from TP_OP_N; footprint TestPoint:TestPoint_Pad_1.0x1.0mm -> TestPoint:TestPoint_Pad_D1.0mm
- TP_OP_OUT1: renamed from TP_OP_OUT; footprint TestPoint:TestPoint_Pad_1.0x1.0mm -> TestPoint:TestPoint_Pad_D1.0mm
- TP_OP_P1: renamed from TP_OP_P; footprint TestPoint:TestPoint_Pad_1.0x1.0mm -> TestPoint:TestPoint_Pad_D1.0mm
- TP_REFp1: footprint TestPoint:TestPoint_THTPad_D1.0mm_Drill0.5mm -> TestPoint:TestPoint_Pad_D1.0mm
Connections:
- net 5V: now also IC1.19 (AVDD_1)
- net Charge-Amplifier-Coarse/Vin_A: now also R14.2
- net Charge-Amplifier-Coarse/Vin_B: now also R18.2
- net Charge-Amplifier-Coarse/Vin_C: now also R21.2
- net Charge-Amplifier-Coarse/Vin_D: now also R22.2
- net Charge-Amplifier-Coarse/Vout_A: now also IC1.2 (IN8P)
- net Charge-Amplifier-Coarse/Vout_B: now also IC1.4 (IN7P)
- net Charge-Amplifier-Coarse/Vout_C: now also IC1.6 (IN6P)
- net Charge-Amplifier-Coarse/Vout_D: now also IC1.8 (IN5P)
- net Charge-Amplifier-Sensitive/Vin_A: now also R23.2
- net Charge-Amplifier-Sensitive/Vin_B: now also R24.2
- net Charge-Amplifier-Sensitive/Vin_C: now also R25.2
- net Charge-Amplifier-Sensitive/Vin_D: now also R26.2
- net Charge-Amplifier-Sensitive/Vout_A: now also IC1.10 (IN4P)
- net Charge-Amplifier-Sensitive/Vout_B: now also IC1.12 (IN3P)
- net Charge-Amplifier-Sensitive/Vout_C: now also IC1.14 (IN2P)
- net Charge-Amplifier-Sensitive/Vout_D: now also IC1.16 (IN1P)
- net GND: now also R5.2, TP_GND1.1; no longer R14.2
- net at R4.2: now also R5.1; no longer R14.1
- net at IC1.44 (GPIO2): now also R1.1; no longer D4.2 (A)
- net ADC.*RESET: now reaches IC1.36 (~{RESET}), J2.1 (Pin_1)
- net at IC1.42 (GPIO1): now also R2.1; no longer D3.2 (A)
- net at IC1.45 (GPIO3): now also D3.2 (A); no longer R2.1
- net at IC1.46 (GPIO4): now also D4.2 (A); no longer R1.1
- new net RJ45-Coarse/A: R14.1
- new net RJ45-Coarse/B: R18.1
- new net RJ45-Coarse/C: R21.1
- new net RJ45-Coarse/D: R22.1
- new net RJ45-Sensitive/A: R23.1
- new net RJ45-Sensitive/B: R24.1
- new net RJ45-Sensitive/C: R25.1
- new net RJ45-Sensitive/D: R26.1
Other:
- removed sheet USB-Connector
- removed sheet USB-Connector1
- removed sheet USB-Connector2
- removed sheet USB-Connector3
- added sheet RJ45-Coarse (RJ45.kicad_sch)
- added sheet RJ45-Sensitive (RJ45.kicad_sch)
- sheet Charge-Amplifier-Coarse ports: added 5V; removed 3.3V
- sheet Charge-Amplifier-Sensitive: file Charge-Amplifier.kicad_sch -> Charge-Amplifier-Sensitive.kicad_sch
- sheet Charge-Amplifier-Sensitive ports: added 5V; removed 3.3V
- note added: "1uF + 100nF for each AVDD/DVDD input -> too much space"
- note added: "Calulation for charge Amplifier: Q=d33*F, Vo = 2V (max. voltage swing) d33 = 500pC/N?, F=1 or 1000N, Cs=20pF?, Rs=100GOhm Vin = Q/Cs Cf = -Q/Vo (feedback Capacitor) fL = 1/(2pi * Rf * Cf) = (Cutoff Frequency)"
- note added: "Input Protection Resistor ! Affects High Frequency FLp = 1 / (2pi * Rin * Cp)"
- note removed: "1uF + 100nF for each AVDD/DVDD input"
- note removed: "R-RJ45R08P-B000? RJ45 Connector Paare: 1+2 3+6 4+5 7+8"
- moved on the sheet: J2

Commit message: updates
Parts:
- added R31: 10k, Resistor_SMD:R_0603_1608Metric, symbol Device:R
- ADC_Daisy1, ADC_TESTN1, ADC_TESTP1, TP_GND1, TP_OP_N1, TP_OP_OUT1, TP_OP_P1, TP_REFp1: footprint TestPoint:TestPoint_Pad_D1.0mm -> TestPoint:TestPoint_Pad_D1.5mm
- J2, J3: footprint Connector_PinHeader_1.00mm:PinHeader_1x02_P1.00mm_Vertical -> Connector_PinHeader_1.27mm:PinHeader_1x02_P1.27mm_Vertical
Connections:
- net 3.3V: now also R31.2
- net at IC1.35 (~{PWDN}), J3.1 (Pin_1): now also R31.1
Other:
- moved on the sheet: J3
Changed lines of the file:
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@@
 	)
 	(junction
+		(at 200.66 123.19)
+		(diameter 0)
+		(color 0 0 0 0)
+	)
+	(junction
 		(at 228.6 21.59)
 		(diameter 0)
@@
 	(wire
 		(pts
+			(xy 200.66 123.19) (xy 200.66 128.27)
+		)
+		(stroke
+			(width 0)
+			(type default)
+		)
+	)
+	(wire
+		(pts
 			(xy 252.73 49.53) (xy 259.08 49.53)
 		)
@@
 	(wire
 		(pts
-			(xy 200.66 114.3) (xy 200.66 120.65)
+			(xy 200.66 114.3) (xy 200.66 123.19)
 		)
 		(stroke
@@
 	)
 	(label "DVDD"
+		(at 208.28 123.19 0)
+		(fields_autoplaced yes)
+		(effects
+			(font
+				(size 1.27 1.27)
+			)
+			(justify left bottom)
+		)
+	)
+	(label "DVDD"
 		(at 170.18 60.96 90)
 		(fields_autoplaced yes)
@@
 			)
 		)
-		(property "Footprint" "TestPoint:TestPoint_Pad_D1.0mm"
+		(property "Footprint" "TestPoint:TestPoint_Pad_D1.5mm"
 			(at 129.54 46.99 0)
 			(effects
@@
 			)
 		)
-		(property "Footprint" "TestPoint:TestPoint_Pad_D1.0mm"
+		(property "Footprint" "TestPoint:TestPoint_Pad_D1.5mm"
 			(at 129.54 41.91 0)
 			(effects
@@
 			)
 		)
-		(property "Footprint" "TestPoint:TestPoint_Pad_D1.0mm"
+		(property "Footprint" "TestPoint:TestPoint_Pad_D1.5mm"
 			(at 180.34 104.14 0)
 			(effects
@@
 			)
 		)
-		(property "Footprint" "TestPoint:TestPoint_Pad_D1.0mm"
+		(property "Footprint" "TestPoint:TestPoint_Pad_D1.5mm"
 			(at 144.78 176.53 0)
 			(effects
@@
 			)
 		)
-		(property "Footprint" "TestPoint:TestPoint_Pad_D1.0mm"
+		(property "Footprint" "TestPoint:TestPoint_Pad_D1.5mm"
 			(at 132.08 137.16 0)
 			(effects
@@
 			)
 		)
-		(property "Footprint" "TestPoint:TestPoint_Pad_D1.0mm"
+		(property "Footprint" "TestPoint:TestPoint_Pad_D1.5mm"
 			(at 129.54 52.07 0)
 			(effects
@@
 	(symbol
 		(lib_id "power:GND")
-		(at 200.66 123.19 270)
+		(at 200.66 130.81 270)
 		(unit 1)
 		(exclude_from_sim no)
@@
 		(fields_autoplaced yes)
 		(property "Reference" "#PWR048"
-			(at 194.31 123.19 0)
+			(at 194.31 130.81 0)
 			(effects
 				(font
@@
 		)
 		(property "Value" "GND"
-			(at 196.85 123.1899 90)
+			(at 196.85 130.8099 90)
 			(effects
 				(font
@@
 		)
 		(property "Footprint" ""
-			(at 200.66 123.19 0)
+			(at 200.66 130.81 0)
 			(effects
 				(font
@@
 		)
 		(property "Datasheet" ""
-			(at 200.66 123.19 0)
+			(at 200.66 130.81 0)
 			(effects
 				(font
@@
 		)
 		(property "Description" "Power symbol creates a global label with name \"GND\" , ground"
-			(at 200.66 123.19 0)
+			(at 200.66 130.81 0)
 			(effects
 				(font
@@
 	)
 	(symbol
+		(lib_id "Device:R")
+		(at 204.47 123.19 90)
+		(unit 1)
+		(exclude_from_sim no)
+		(in_bom yes)
+		(on_board yes)
+		(dnp no)
+		(property "Reference" "R31"
+			(at 218.186 121.92 90)
+			(effects
+				(font
+					(size 1.27 1.27)
+				)
+				(hide yes)
+			)
+		)
+		(property "Value" "10k"
+			(at 204.47 125.222 90)
+			(effects
+				(font
+					(size 1.27 1.27)
+				)
+			)
+		)
+		(property "Footprint" "Resistor_SMD:R_0603_1608Metric"
+			(at 204.47 124.968 90)
+			(effects
+				(font
+					(size 1.27 1.27)
+				)
+				(hide yes)
+			)
+		)
+		(property "Datasheet" "~"
+			(at 204.47 123.19 0)
+			(effects
+				(font
+					(size 1.27 1.27)
+				)
+				(hide yes)
+			)
+		)
+		(property "Description" "Resistor"
+			(at 204.47 123.19 0)
+			(effects
+				(font
+					(size 1.27 1.27)
+				)
+				(hide yes)
+			)
+		)
+		(pin "2"
+		)
+		(pin "1"
+		)
+		(instances
+			(project "Schlaubi-Schlumpf"
+				(path "/adec948c-82e6-4ad4-8e75-b19e612c0d17/2131c80a-ce05-49b0-92ac-52a13fef390c"
+					(reference "R31")
+					(unit 1)
+				)
+			)
+		)
+	)
+	(symbol
 		(lib_id "power:GND")
 		(at 119.38 163.83 0)
@@
 			)
 		)
-		(property "Footprint" "TestPoint:TestPoint_Pad_D1.0mm"
+		(property "Footprint" "TestPoint:TestPoint_Pad_D1.5mm"
 			(at 124.46 163.83 0)
 			(effects
@@
 	(symbol
 		(lib_id "Connector:Conn_01x02_Pin")
-		(at 205.74 120.65 0)
+		(at 205.74 128.27 0)
 		(mirror y)
 		(unit 1)
@@
 		(dnp no)
 		(property "Reference" "J3"
-			(at 207.01 123.1901 0)
+			(at 207.01 130.8101 0)
 			(effects
 				(font
@@
 		)
 		(property "Value" "Conn_01x02_Pin"
-			(at 207.01 120.6501 0)
+			(at 207.01 128.2701 0)
 			(effects
 				(font
@@
 			)
 		)
-		(property "Footprint" "Connector_PinHeader_1.00mm:PinHeader_1x02_P1.00mm_Vertical"
-			(at 205.74 120.65 0)
+		(property "Footprint" "Connector_PinHeader_1.27mm:PinHeader_1x02_P1.27mm_Vertical"
+			(at 205.74 128.27 0)
 			(effects
 				(font
@@
 		)
 		(property "Datasheet" "~"
-			(at 205.74 120.65 0)
+			(at 205.74 128.27 0)
 			(effects
 				(font
@@
 		)
 		(property "Description" "Generic connector, single row, 01x02, script generated"
-			(at 205.74 120.65 0)
+			(at 205.74 128.27 0)
 			(effects
 				(font
@@
 			)
 		)
-		(property "Footprint" "TestPoint:TestPoint_Pad_D1.0mm"
+		(property "Footprint" "TestPoint:TestPoint_Pad_D1.5mm"
 			(at 129.54 137.16 0)
 			(effects
@@
 			)
 		)
-		(property "Footprint" "Connector_PinHeader_1.00mm:PinHeader_1x02_P1.00mm_Vertical"
+		(property "Footprint" "Connector_PinHeader_1.27mm:PinHeader_1x02_P1.27mm_Vertical"
 			(at 210.82 111.76 0)
 			(effects

Commit message: update Opamp
Parts:
- removed R14, R18, R21, R22, R23, R24, R25, R26: 0R, Resistor_SMD:R_0603_1608Metric, symbol Device:R
- added CS15: 100n, Capacitor_SMD:C_0603_1608Metric, symbol Device:C
- added IC3: TLV9051IDBVR, TLV9051IDBVR:SOT95P280X145-5N, symbol TLV9051IDBVR:TLV9051IDBVR
- added Rf_Opamp1: 0R, Resistor_SMD:R_0603_1608Metric, symbol Device:R
- added TP_SHIELD1, TP_VBIAS1: TestPoint, TestPoint:TestPoint_Pad_D1.5mm, symbol Connector:TestPoint
Connections:
- net GND: now also CS15.2, IC3.2 (V-); no longer IC1.1 (IN8N), IC1.11 (IN3N), IC1.13 (IN2N), IC1.15 (IN1N), IC1.3 (IN7N), IC1.5 (IN6N), IC1.7 (IN5N), IC1.9 (IN4N)
- net at IC1.61 (OPAMPN), TP_OP_N1.1: now also Rf_Opamp1.2
- net at IC1.63 (OPAMPOUT), TP_OP_OUT1.1: now also IC3.3 (IN+), Rf_Opamp1.1
- net ADC.*PWDN: now reaches IC1.35 (~{PWDN}), J3.1 (Pin_1), R31.1
- new net Shield: TP_SHIELD1.1
- new net Vbias: IC1.1 (IN8N), IC1.11 (IN3N), IC1.13 (IN2N), IC1.15 (IN1N), IC1.3 (IN7N), IC1.5 (IN6N), IC1.7 (IN5N), IC1.9 (IN4N), IC3.1 (OUT), IC3.4 (IN-), TP_VBIAS1.1
- new net non_reg: CS15.1, IC3.5 (V+)
Other:
- sheet Charge-Amplifier-Coarse ports: added Vbias; removed Vref
- sheet Charge-Amplifier-Sensitive ports: added Vbias; removed Vref
- sheet RJ45-Coarse ports: added Vbias; removed Vref
- sheet RJ45-Sensitive ports: added Vbias; removed Vref
- note added: "Programming: - Set SPI Mode (0,1) CPOL=0, CPHA=1 - (VREF_4V <= 1) Set internal Reference Voltage to 4V - (OPAMP_REF <= 1) Set Opamp reference to (AVDD+AVSS) / 2"
- note added: "internal Opamp (AVDD+AVSS)/2 = Vbias ! Set OPAMP_REF <= 1"
- note removed: "Programming: - Set SPI Mode (0,1) CPOL=0, CPHA=1 - Set internal Reference Voltage to 4V"
- note removed: "use internal opamp + unity gain buffer for OP-Amp Bias"
- moved on the sheet: TP_GND1, TP_OP_N1, TP_OP_OUT1, TP_OP_P1

Commit message: newest order 17.09
Parts:
- removed R31: 10k, Resistor_SMD:R_0603_1608Metric, symbol Device:R
- ADC_Daisy1, ADC_TESTN1, ADC_TESTP1, TP_GND1, TP_OP_N1, TP_OP_OUT1, TP_OP_P1, TP_REFp1, TP_SHIELD1, TP_VBIAS1: footprint TestPoint:TestPoint_Pad_D1.5mm -> TestPoint:TestPoint_Pad_D1.0mm
Other:
- note added: "Programming: - Set *RESET and *PWDN to High - Set SPI Mode (0,1) CPOL=0, CPHA=1 - (VREF_4V <= 1) Set internal Reference Voltage to 4V - (OPAMP_REF <= 1) Set Opamp reference to (AVDD+AVSS) / 2"
- note removed: "Programming: - Set SPI Mode (0,1) CPOL=0, CPHA=1 - (VREF_4V <= 1) Set internal Reference Voltage to 4V - (OPAMP_REF <= 1) Set Opamp reference to (AVDD+AVSS) / 2"
