File: PCB/Schlaubi-Schlumpf/Charge-Amplifier-Sensitive.kicad_sch (KiCad schematic)
At the start: 13 parts, among them U1 AD8608ARUZ-REEL

Commit message: update Opamp
Parts:
- CF1, CF2, CF3, CF4: footprint Capacitor_SMD:C_0603_1608Metric -> Capacitor_SMD:C_0805_2012Metric_Pad1.18x1.45mm_HandSolder
- RF1, RF2, RF3, RF4: footprint Resistor_SMD:R_0805_2012Metric -> Resistor_SMD:R_0805_2012Metric_Pad1.20x1.40mm_HandSolder
Connections:
- net Vref renamed Vbias
Changed lines of the file:
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@@
 		)
 	)
-	(hierarchical_label "Vref"
+	(hierarchical_label "Vbias"
 		(shape input)
-		(at 107.95 87.63 180)
+		(at 107.95 82.55 180)
 		(fields_autoplaced yes)
 		(effects
@@
 		)
 	)
-	(hierarchical_label "Vref"
+	(hierarchical_label "Vbias"
 		(shape input)
-		(at 194.31 87.63 0)
-		(fields_autoplaced yes)
-		(effects
-			(font
-				(size 1.27 1.27)
-			)
-			(justify left)
+		(at 107.95 87.63 180)
+		(fields_autoplaced yes)
+		(effects
+			(font
+				(size 1.27 1.27)
+			)
+			(justify right)
 		)
 	)
@@
 		)
 	)
+	(hierarchical_label "Vbias"
+		(shape input)
+		(at 138.43 105.41 180)
+		(fields_autoplaced yes)
+		(effects
+			(font
+				(size 1.27 1.27)
+			)
+			(justify right)
+		)
+	)
 	(hierarchical_label "Vin_C"
 		(shape input)
@@
 		)
 	)
-	(hierarchical_label "Vref"
+	(hierarchical_label "Vbias"
 		(shape input)
 		(at 194.31 82.55 0)
@@
 			)
 			(justify left)
-		)
-	)
-	(hierarchical_label "Vref"
-		(shape input)
-		(at 138.43 105.41 180)
-		(fields_autoplaced yes)
-		(effects
-			(font
-				(size 1.27 1.27)
-			)
-			(justify right)
 		)
 	)
@@
 		)
 	)
-	(hierarchical_label "Vref"
-		(shape input)
-		(at 107.95 82.55 180)
-		(fields_autoplaced yes)
-		(effects
-			(font
-				(size 1.27 1.27)
-			)
-			(justify right)
-		)
-	)
 	(hierarchical_label "Vout_C"
 		(shape output)
@@
 		)
 	)
+	(hierarchical_label "Vbias"
+		(shape input)
+		(at 194.31 87.63 0)
+		(fields_autoplaced yes)
+		(effects
+			(font
+				(size 1.27 1.27)
+			)
+			(justify left)
+		)
+	)
 	(symbol
 		(lib_id "power:GND")
@@
 			)
 		)
-		(property "Footprint" "Resistor_SMD:R_0805_2012Metric"
+		(property "Footprint" "Resistor_SMD:R_0805_2012Metric_Pad1.20x1.40mm_HandSolder"
 			(at 183.642 93.98 90)
 			(effects
@@
 			)
 		)
-		(property "Footprint" "Resistor_SMD:R_0805_2012Metric"
+		(property "Footprint" "Resistor_SMD:R_0805_2012Metric_Pad1.20x1.40mm_HandSolder"
 			(at 183.642 76.2 90)
 			(effects
@@
 			)
 		)
-		(property "Footprint" "Resistor_SMD:R_0805_2012Metric"
+		(property "Footprint" "Resistor_SMD:R_0805_2012Metric_Pad1.20x1.40mm_HandSolder"
 			(at 121.412 76.2 90)
 			(effects
@@
 			)
 		)
-		(property "Footprint" "Capacitor_SMD:C_0603_1608Metric"
+		(property "Footprint" "Capacitor_SMD:C_0805_2012Metric_Pad1.18x1.45mm_HandSolder"
 			(at 181.3052 97.79 0)
 			(effects
@@
 			)
 		)
-		(property "Footprint" "Resistor_SMD:R_0805_2012Metric"
+		(property "Footprint" "Resistor_SMD:R_0805_2012Metric_Pad1.20x1.40mm_HandSolder"
 			(at 121.412 93.98 90)
 			(effects
@@
 			)
 		)
-		(property "Footprint" "Capacitor_SMD:C_0603_1608Metric"
+		(property "Footprint" "Capacitor_SMD:C_0805_2012Metric_Pad1.18x1.45mm_HandSolder"
 			(at 119.0752 97.79 0)
 			(effects
@@
 			)
 		)
-		(property "Footprint" "Capacitor_SMD:C_0603_1608Metric"
+		(property "Footprint" "Capacitor_SMD:C_0805_2012Metric_Pad1.18x1.45mm_HandSolder"
 			(at 181.3052 80.01 0)
 			(effects
@@
 			)
 		)
-		(property "Footprint" "Capacitor_SMD:C_0603_1608Metric"
+		(property "Footprint" "Capacitor_SMD:C_0805_2012Metric_Pad1.18x1.45mm_HandSolder"
 			(at 119.0752 80.01 0)
 			(effects

Commit message: newest order 17.09
Parts:
- CF1, CF2, CF3, CF4: value 330p -> 680p
- RF1, RF2, RF3, RF4: value 2G -> 1G
Changed lines of the file:
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@@
 (kicad_sch
-	(version 20231120)
+	(version 20250114)
 	(generator "eeschema")
-	(generator_version "8.0")
+	(generator_version "9.0")
 	(paper "A4")
 	(junction
@@
 		(shape input)
 		(at 107.95 82.55 180)
-		(fields_autoplaced yes)
 		(effects
 			(font
@@
 		(shape input)
 		(at 107.95 80.01 180)
-		(fields_autoplaced yes)
 		(effects
 			(font
@@
 		(shape input)
 		(at 107.95 87.63 180)
-		(fields_autoplaced yes)
 		(effects
 			(font
@@
 		(shape input)
 		(at 107.95 90.17 180)
-		(fields_autoplaced yes)
 		(effects
 			(font
@@
 		(shape input)
 		(at 194.31 80.01 0)
-		(fields_autoplaced yes)
 		(effects
 			(font
@@
 		(shape input)
 		(at 138.43 105.41 180)
-		(fields_autoplaced yes)
 		(effects
 			(font
@@
 		(shape input)
 		(at 194.31 90.17 0)
-		(fields_autoplaced yes)
 		(effects
 			(font
@@
 		(shape output)
 		(at 107.95 72.39 180)
-		(fields_autoplaced yes)
 		(effects
 			(font
@@
 		(shape input)
 		(at 194.31 82.55 0)
-		(fields_autoplaced yes)
 		(effects
 			(font
@@
 		(shape output)
 		(at 194.31 72.39 0)
-		(fields_autoplaced yes)
 		(effects
 			(font
@@
 		(shape input)
 		(at 73.66 85.09 180)
-		(fields_autoplaced yes)
 		(effects
 			(font
@@
 		(shape output)
 		(at 107.95 97.79 180)
-		(fields_autoplaced yes)
 		(effects
 			(font
@@
 		(shape output)
 		(at 194.31 97.79 0)
-		(fields_autoplaced yes)
 		(effects
 			(font
@@
 		(shape input)
 		(at 194.31 87.63 0)
-		(fields_autoplaced yes)
 		(effects
 			(font
@@
 			)
 		)
-		(property "Value" "2G"
+		(property "Value" "1G"
 			(at 187.96 95.2499 0)
 			(effects
@@
 			)
 		)
-		(property "Value" "2G"
+		(property "Value" "1G"
 			(at 187.96 77.4699 0)
 			(effects
@@
 			)
 		)
-		(property "Value" "2G"
+		(property "Value" "1G"
 			(at 125.73 77.4699 0)
 			(effects
@@
 			)
 		)
-		(property "Value" "330p"
+		(property "Value" "680p"
 			(at 172.974 94.488 0)
 			(effects
@@
 			)
 		)
-		(property "Value" "2G"
+		(property "Value" "1G"
 			(at 125.73 95.2499 0)
 			(effects
@@
 			)
 		)
-		(property "Value" "330p"
+		(property "Value" "680p"
 			(at 110.744 94.488 0)
 			(effects
@@
 			)
 		)
-		(property "Value" "330p"
+		(property "Value" "680p"
 			(at 172.974 76.708 0)
 			(effects
@@
 			)
 		)
-		(property "Value" "330p"
+		(property "Value" "680p"
 			(at 110.744 76.708 0)
 			(effects
