File: PCB/Schlaubi-Schlumpf/Charge-Amplifier.kicad_sch (KiCad schematic)
At the start: 13 parts, among them U1 AD8608ARUZ-REEL

Commit message: v1
Parts:
- removed CF1, CF2, CF3, CF4: 360p, Capacitor_SMD:C_0603_1608Metric, symbol Device:C
- removed CS16, CS18: 10u, Capacitor_SMD:C_0603_1608Metric, symbol Device:C
- removed CS17, CS19: 100n, Capacitor_SMD:C_0603_1608Metric, symbol Device:C
- removed RF1, RF2, RF3, RF4: 2G, Resistor_SMD:R_0603_1608Metric, symbol Device:R
- removed U1: AD8608ARUZ-REEL, AD8608ARUZ:RU_14_ADI, symbol AD8608ARUZ:AD8608ARUZ-REEL
- added CF5, CF6, CF7, CF8: 330n, Capacitor_SMD:C_0603_1608Metric, symbol Device:C
- added CS50, CS52: 10u, Capacitor_SMD:C_0603_1608Metric, symbol Device:C
- added CS51, CS53: 100n, Capacitor_SMD:C_0603_1608Metric, symbol Device:C
- added RF5, RF6, RF7, RF8: 15k, Resistor_SMD:R_0603_1608Metric, symbol Device:R
- added U4: AD8608ARUZ-REEL, AD8608ARUZ:RU_14_ADI, symbol AD8608ARUZ:AD8608ARUZ-REEL
Connections:
- net GND: now also CS50.2, CS51.2, CS52.2, CS53.2, U4.11 (V-)
- net Vin_A: now also CF5.2, RF5.2, U4.2 (-INA)
- net Vin_B: now also CF6.1, RF6.1, U4.6 (-INB)
- net Vin_C: now also CF8.1, RF8.1, U4.9 (-INC)
- net Vin_D: now also CF7.2, RF7.2, U4.13 (-IND)
- net Vout_A: now also CF5.1, RF5.1, U4.1 (OUTA)
- net Vout_B: now also CF6.2, RF6.2, U4.7 (OUTB)
- net Vout_C: now also CF8.2, RF8.2, U4.8 (OUTC)
- net Vout_D: now also CF7.1, RF7.1, U4.14 (OUTD)
- net Vref: now also CS52.1, CS53.1, U4.10 (+INC), U4.12 (+IND), U4.3 (+INA), U4.5 (+INB)
- new net 5V: CS50.1, CS51.1, U4.4 (V+)

Commit message: updates
Parts:
- RF5, RF6, RF7, RF8: footprint Resistor_SMD:R_0603_1608Metric -> Resistor_SMD:R_0805_2012Metric
Changed lines of the file:
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@@
 			)
 		)
-		(property "Footprint" "Resistor_SMD:R_0603_1608Metric"
+		(property "Footprint" "Resistor_SMD:R_0805_2012Metric"
 			(at 183.642 93.98 90)
 			(effects
@@
 			)
 		)
-		(property "Footprint" "Resistor_SMD:R_0603_1608Metric"
+		(property "Footprint" "Resistor_SMD:R_0805_2012Metric"
 			(at 121.412 76.2 90)
 			(effects
@@
 			)
 		)
-		(property "Footprint" "Resistor_SMD:R_0603_1608Metric"
+		(property "Footprint" "Resistor_SMD:R_0805_2012Metric"
 			(at 183.642 76.2 90)
 			(effects
@@
 			)
 		)
-		(property "Footprint" "Resistor_SMD:R_0603_1608Metric"
+		(property "Footprint" "Resistor_SMD:R_0805_2012Metric"
 			(at 121.412 93.98 90)
 			(effects

Commit message: update Opamp
Parts:
- CF5, CF6, CF7, CF8: footprint Capacitor_SMD:C_0603_1608Metric -> Capacitor_SMD:C_0805_2012Metric_Pad1.18x1.45mm_HandSolder
- RF5, RF6, RF7, RF8: footprint Resistor_SMD:R_0805_2012Metric -> Resistor_SMD:R_0805_2012Metric_Pad1.20x1.40mm_HandSolder
Connections:
- net Vref renamed Vbias
Changed lines of the file:
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@@
+		)
+	)
+	(hierarchical_label "Vbias"
+		(shape input)
+		(at 138.43 105.41 180)
+		(fields_autoplaced yes)
+		(effects
+			(font
+				(size 1.27 1.27)
+			)
+			(justify right)
 		)
 	)
@@
 		)
 	)
-	(hierarchical_label "Vref"
+	(hierarchical_label "Vbias"
 		(shape input)
-		(at 107.95 82.55 180)
-		(fields_autoplaced yes)
-		(effects
-			(font
-				(size 1.27 1.27)
-			)
-			(justify right)
+		(at 194.31 87.63 0)
+		(fields_autoplaced yes)
+		(effects
+			(font
+				(size 1.27 1.27)
+			)
+			(justify left)
 		)
 	)
@@
 		)
 	)
-	(hierarchical_label "Vref"
+	(hierarchical_label "Vbias"
 		(shape input)
-		(at 138.43 105.41 180)
+		(at 107.95 82.55 180)
 		(fields_autoplaced yes)
 		(effects
@@
 		)
 	)
-	(hierarchical_label "Vref"
+	(hierarchical_label "Vbias"
+		(shape input)
+		(at 107.95 87.63 180)
+		(fields_autoplaced yes)
+		(effects
+			(font
+				(size 1.27 1.27)
+			)
+			(justify right)
+		)
+	)
+	(hierarchical_label "Vbias"
 		(shape input)
 		(at 194.31 82.55 0)
@@
 		)
 	)
-	(hierarchical_label "Vref"
-		(shape input)
-		(at 107.95 87.63 180)
-		(fields_autoplaced yes)
-		(effects
-			(font
-				(size 1.27 1.27)
-			)
-			(justify right)
-		)
-	)
 	(hierarchical_label "Vin_A"
 		(shape input)
@@
 		)
 	)
-	(hierarchical_label "Vref"
-		(shape input)
-		(at 194.31 87.63 0)
-		(fields_autoplaced yes)
-		(effects
-			(font
-				(size 1.27 1.27)
-			)
-			(justify left)
-		)
-	)
 	(hierarchical_label "5V"
 		(shape input)
@@
 			)
 		)
-		(property "Footprint" "Resistor_SMD:R_0805_2012Metric"
+		(property "Footprint" "Resistor_SMD:R_0805_2012Metric_Pad1.20x1.40mm_HandSolder"
 			(at 183.642 93.98 90)
 			(effects
@@
 			)
 		)
-		(property "Footprint" "Resistor_SMD:R_0805_2012Metric"
+		(property "Footprint" "Resistor_SMD:R_0805_2012Metric_Pad1.20x1.40mm_HandSolder"
 			(at 121.412 76.2 90)
 			(effects
@@
 			)
 		)
-		(property "Footprint" "Resistor_SMD:R_0805_2012Metric"
+		(property "Footprint" "Resistor_SMD:R_0805_2012Metric_Pad1.20x1.40mm_HandSolder"
 			(at 183.642 76.2 90)
 			(effects
@@
 			)
 		)
-		(property "Footprint" "Capacitor_SMD:C_0603_1608Metric"
+		(property "Footprint" "Capacitor_SMD:C_0805_2012Metric_Pad1.18x1.45mm_HandSolder"
 			(at 119.0752 97.79 0)
 			(effects
@@
 			)
 		)
-		(property "Footprint" "Capacitor_SMD:C_0603_1608Metric"
+		(property "Footprint" "Capacitor_SMD:C_0805_2012Metric_Pad1.18x1.45mm_HandSolder"
 			(at 181.3052 97.79 0)
 			(effects
@@
 			)
 		)
-		(property "Footprint" "Capacitor_SMD:C_0603_1608Metric"
+		(property "Footprint" "Capacitor_SMD:C_0805_2012Metric_Pad1.18x1.45mm_HandSolder"
 			(at 119.0752 80.01 0)
 			(effects
@@
 			)
 		)
-		(property "Footprint" "Capacitor_SMD:C_0603_1608Metric"
+		(property "Footprint" "Capacitor_SMD:C_0805_2012Metric_Pad1.18x1.45mm_HandSolder"
 			(at 181.3052 80.01 0)
 			(effects
@@
 			)
 		)
-		(property "Footprint" "Resistor_SMD:R_0805_2012Metric"
+		(property "Footprint" "Resistor_SMD:R_0805_2012Metric_Pad1.20x1.40mm_HandSolder"
 			(at 121.412 93.98 90)
 			(effects

Commit message: newest order 17.09
Parts:
- CF5, CF6, CF7, CF8: value 330n -> 680p
- RF5, RF6, RF7, RF8: value 15k -> 1G
Changed lines of the file:
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@@
 (kicad_sch
-	(version 20231120)
+	(version 20250114)
 	(generator "eeschema")
-	(generator_version "8.0")
+	(generator_version "9.0")
 	(paper "A4")
 	(junction
@@
 		(shape input)
 		(at 138.43 105.41 180)
-		(fields_autoplaced yes)
 		(effects
 			(font
@@
 		(shape output)
 		(at 107.95 72.39 180)
-		(fields_autoplaced yes)
 		(effects
 			(font
@@
 		(shape input)
 		(at 194.31 87.63 0)
-		(fields_autoplaced yes)
 		(effects
 			(font
@@
 		(shape input)
 		(at 107.95 90.17 180)
-		(fields_autoplaced yes)
 		(effects
 			(font
@@
 		(shape output)
 		(at 194.31 97.79 0)
-		(fields_autoplaced yes)
 		(effects
 			(font
@@
 		(shape output)
 		(at 107.95 97.79 180)
-		(fields_autoplaced yes)
 		(effects
 			(font
@@
 		(shape input)
 		(at 107.95 82.55 180)
-		(fields_autoplaced yes)
 		(effects
 			(font
@@
 		(shape input)
 		(at 107.95 87.63 180)
-		(fields_autoplaced yes)
 		(effects
 			(font
@@
 		(shape input)
 		(at 194.31 82.55 0)
-		(fields_autoplaced yes)
 		(effects
 			(font
@@
 		(shape input)
 		(at 194.31 90.17 0)
-		(fields_autoplaced yes)
 		(effects
 			(font
@@
 		(shape input)
 		(at 107.95 80.01 180)
-		(fields_autoplaced yes)
 		(effects
 			(font
@@
 		(shape input)
 		(at 73.66 85.09 180)
-		(fields_autoplaced yes)
 		(effects
 			(font
@@
 		(shape output)
 		(at 194.31 72.39 0)
-		(fields_autoplaced yes)
 		(effects
 			(font
@@
 		(shape input)
 		(at 194.31 80.01 0)
-		(fields_autoplaced yes)
 		(effects
 			(font
@@
 			)
 		)
-		(property "Value" "15k"
+		(property "Value" "1G"
 			(at 187.96 95.2499 0)
 			(effects
@@
 		(fields_autoplaced yes)
 		(property "Reference" "RF5"
-			(at 125.73 75.5649 0)
-			(effects
-				(font
-					(size 1.27 1.27)
-				)
-				(justify left)
-			)
-		)
-		(property "Value" "15k"
-			(at 125.73 77.47 0)
+			(at 125.73 74.9299 0)
+			(effects
+				(font
+					(size 1.27 1.27)
+				)
+				(justify left)
+			)
+		)
+		(property "Value" "1G"
+			(at 125.73 77.4699 0)
 			(effects
 				(font
@@
 			)
 		)
-		(property "Value" "15k"
+		(property "Value" "1G"
 			(at 187.96 77.4699 0)
 			(effects
@@
 			)
 		)
-		(property "Value" "330n"
+		(property "Value" "680p"
 			(at 110.744 94.488 0)
 			(effects
@@
 			)
 		)
-		(property "Value" "330n"
+		(property "Value" "680p"
 			(at 172.974 94.488 0)
 			(effects
@@
 			)
 		)
-		(property "Value" "330n"
+		(property "Value" "680p"
 			(at 110.744 76.708 0)
 			(effects
@@
 			)
 		)
-		(property "Value" "330n"
+		(property "Value" "680p"
 			(at 172.974 76.708 0)
 			(effects
@@
 			)
 		)
-		(property "Value" "15k"
+		(property "Value" "1G"
 			(at 125.73 95.2499 0)
 			(effects
