File: PCB/Schlaubi-Schlumpf/RJ45.kicad_sch (KiCad schematic)
At the start: 1 part, among them J5 8P8C_Shielded

Commit message: update Opamp
Connections:
- net Vref renamed Vbias
Changed lines of the file:
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@@
 		)
 	)
-	(hierarchical_label "B"
-		(shape output)
-		(at 135.89 86.36 0)
-		(fields_autoplaced yes)
-		(effects
-			(font
-				(size 1.27 1.27)
-			)
-			(justify left)
-		)
-	)
-	(hierarchical_label "Vref"
+	(hierarchical_label "Vbias"
 		(shape input)
 		(at 135.89 88.9 0)
@@
 		)
 	)
-	(hierarchical_label "Vref"
-		(shape input)
-		(at 135.89 81.28 0)
+	(hierarchical_label "B"
+		(shape output)
+		(at 135.89 86.36 0)
 		(fields_autoplaced yes)
 		(effects
@@
 		)
 	)
-	(hierarchical_label "Vref"
+	(hierarchical_label "Vbias"
 		(shape input)
-		(at 135.89 73.66 0)
+		(at 135.89 83.82 0)
 		(fields_autoplaced yes)
 		(effects
@@
 		)
 	)
-	(hierarchical_label "Vref"
+	(hierarchical_label "Vbias"
 		(shape input)
-		(at 135.89 83.82 0)
+		(at 135.89 81.28 0)
 		(fields_autoplaced yes)
 		(effects
@@
 		(fields_autoplaced yes)
 		(effects
+			(font
+				(size 1.27 1.27)
+			)
+			(justify left)
+		)
+	)
+	(hierarchical_label "Vbias"
+		(shape input)
+		(at 135.89 73.66 0)
+		(fields_autoplaced yes)
+		(effects

Commit message: newest order 17.09
Parts:
- renumbered J5 to J1
Changed lines of the file:
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@@
 (kicad_sch
-	(version 20231120)
+	(version 20250114)
 	(generator "eeschema")
-	(generator_version "8.0")
+	(generator_version "9.0")
 	(paper "A4")
-	(wire
-		(pts
-			(xy 125.73 95.25) (xy 125.73 93.98)
-		)
-		(stroke
-			(width 0)
-			(type default)
-		)
-	)
 	(text "R-RJ45R08P-B000?\nRJ45 Connector pairs -> T-568B standard:\n-> higher number is full color, lower striped\n1+2 orange/B\n3+6 green/C\n4+5 blue/A\n7+8 brown/D\n"
 		(exclude_from_sim no)
@@
 			)
 			(justify left)
+		)
+	)
+	(wire
+		(pts
+			(xy 125.73 95.25) (xy 125.73 93.98)
+		)
+		(stroke
+			(width 0)
+			(type default)
 		)
 	)
@@
 		(shape input)
 		(at 135.89 88.9 0)
-		(fields_autoplaced yes)
 		(effects
 			(font
@@
 		(shape output)
 		(at 135.89 86.36 0)
-		(fields_autoplaced yes)
 		(effects
 			(font
@@
 		(shape output)
 		(at 135.89 78.74 0)
-		(fields_autoplaced yes)
 		(effects
 			(font
@@
 		(shape input)
 		(at 135.89 83.82 0)
-		(fields_autoplaced yes)
 		(effects
 			(font
@@
 		(shape output)
 		(at 135.89 71.12 0)
-		(fields_autoplaced yes)
 		(effects
 			(font
@@
 		(shape input)
 		(at 135.89 81.28 0)
-		(fields_autoplaced yes)
 		(effects
 			(font
@@
 		(shape output)
 		(at 135.89 76.2 0)
-		(fields_autoplaced yes)
 		(effects
 			(font
@@
 		(shape input)
 		(at 135.89 73.66 0)
-		(fields_autoplaced yes)
 		(effects
 			(font
@@
 		(dnp no)
 		(fields_autoplaced yes)
-		(property "Reference" "J5"
+		(property "Reference" "J1"
 			(at 125.73 63.5 0)
 			(effects
