File: PCB/Schlaubi-Schlumpf/Schlaubi-Schlumpf.kicad_pcb (KiCad board)
At the start: 4 copper layers, 50 x 67 mm, 150 parts, among them IC1 ADS131E08IPAGR, IC2 TP4056, IC3 TPS7A8801RTJR, IC7 LM2775QDSGRQ1, J1 8P8C_Shielded, J2 Conn_01x02_Pin, J3 Conn_01x02_Pin, J4 Conn_01x02_Pin, J5 8P8C_Shielded, J6 TYPE-C-31-M-12, J7 RFShield_TwoPieces, Q1 DMG2305, U1 AD8608ARUZ-REEL, U2 ESP32-S3-MINI-1-N8, U3 ICM-42670-P, U4 AD8608ARUZ-REEL

Commit message: updates
Parts:
- removed H1, H3: MountingHole_Pad, MountingHole:MountingHole_3.2mm_M3_Pad
- added R31: 10k, Resistor_SMD:R_0603_1608Metric, F.Cu at (77.5, 68.0)
- CS22, CS23: value 10n -> 100n
- GPIO2, GPIO3, J2, J3, UART0, UART1: footprint Connector_PinHeader_1.00mm:PinHeader_1x02_P1.00mm_Vertical -> Connector_PinHeader_1.27mm:PinHeader_1x02_P1.27mm_Vertical
- RF5, RF6, RF7, RF8: footprint Resistor_SMD:R_0603_1608Metric -> Resistor_SMD:R_0805_2012Metric
- SPIEXT1: footprint Connector_PinHeader_1.00mm:PinHeader_1x04_P1.00mm_Vertical -> Connector_PinHeader_1.27mm:PinHeader_1x04_P1.27mm_Vertical
- TP_OP_OUT1, TP_REFp1: moved to B.Cu
- moved G*** 65.5 mm to (120.8, 91.7)
- moved JP1 44.5 mm to (120.8, 57.4), turned to -90 degrees
- moved H2 43.2 mm to (112.1, 58.6)
- moved CCHARGE1 41.6 mm to (117.7, 55.6), turned to 0 degrees
- moved CS40 40.7 mm to (117.7, 60.6), turned to 0 degrees
- moved IC7 39.4 mm to (117.7, 58.0), turned to -90 degrees
- moved CS44 38.9 mm to (117.7, 62.1), turned to 0 degrees
- moved CS41 38.2 mm to (120.7, 60.6), turned to 0 degrees
- moved CS43 37.3 mm to (120.7, 62.1), turned to 0 degrees
- moved J2 14.0 mm to (75.4, 64.8)
- moved CS20 11.7 mm to (100.9, 57.7), turned to 0 degrees
- moved CS21 11.1 mm to (97.9, 57.7), turned to 0 degrees
- moved J3 8.95 mm to (75.3, 68.0), turned to -90 degrees
- moved J5 8.06 mm to (116.6, 90.0)
- moved J1 8.06 mm to (116.6, 69.8)
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Connections:
- J4 pad 1: GND -> /Power_battery/Bat+
- J4 pad 2: /Power_battery/Bat+ -> GND
Routing:
- net /Power_battery/non_reg_in: track 102.3 -> 54.3 mm
- net /ADC/AVDD: track 99.8 -> 137.1 mm
- net Shield: track 26.9 -> 0.00 mm, vias 48 -> 42
- net /ADC/RJ45-Coarse/B: track 28.1 -> 15.5 mm, vias 0 -> 1
- net /ADC/ADC.*RESET: track 33.4 -> 44.9 mm
- net Net-(IC1-~{PWDN}): track 18.9 -> 28.3 mm
- net /ADC/Vref: track 130.1 -> 121.2 mm
- net GND: track 123.1 -> 115.3 mm, vias 110 -> 111
- net /ADC/RJ45-Sensitive/B: track 31.5 -> 25.9 mm
- net /ADC/RJ45-Sensitive/A: track 24.5 -> 19.2 mm
- net /Power_battery/Bat+: track 21.6 -> 26.3 mm
- net /ADC/RJ45-Sensitive/C: track 17.6 -> 13.7 mm
- net /ESP32/U1TXD: track 2.29 -> 5.43 mm
- net /ADC/DVDD: track 143.6 -> 146.3 mm, vias 7 -> 9
- net /ESP32/IMU.CS: track 6.50 -> 9.01 mm
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Other:
- board size 50 x 67 mm -> 50 x 65 mm
- board text added: "*PWDN"
- board text added: "*RESET"
- board text added: "1"
- board text added: "2"
- board text added: "3"
- board text added: "4"
- board text added: "5"
- board text added: "6"
- board text added: "7"
- board text added: "8"
- board text added: "BATTERY"
- board text added: "BOOT"
- board text added: "Bat+"
- board text added: "GPIO2"
- board text added: "GPIO3"
- board text added: "PINOUT ADC IN8 - A_coarse IN7 - B_coarse IN6 - C_coarse IN5 - D_coarse IN4 - A_sensitive IN3 - B_sensitive IN2 - C_sensitive IN1 - D_sensitive"
- board text added: "PINOUT RJ45 (T-568B) 1+2 orange/B 3+6 green/C 4+5 blue/A 7+8 brown/D (striped + full) (Vref+Pin)"
- board text added: "Schlaubi-Schlumpf v1.0 (Multi-Ferro-DAQ) Mark Suppelt"
- board text added: "striped (1,3,4,7) on Vref"
- board text removed: "IO GND"
- board text removed: "Schlaubi-Schlumpf (Multi-Ferro-DAQ) Mark Suppelt"

Commit message: update Opamp
Parts:
- removed CS20, CS21, CS26, CS27: 10u, Capacitor_SMD:C_0603_1608Metric
- removed CS22, CS23: 100n, Capacitor_SMD:C_0603_1608Metric
- removed CS24, CS25: 10n, Capacitor_SMD:C_0603_1608Metric
- removed R10: 15k, Resistor_SMD:R_0603_1608Metric
- removed R11: 10k, Resistor_SMD:R_0603_1608Metric
- removed R14, R18, R21, R22, R23, R24, R25, R26: 0R, Resistor_SMD:R_0603_1608Metric
- removed R8: 1.15k, Resistor_SMD:R_0603_1608Metric
- removed R9: 3.57k, Resistor_SMD:R_0603_1608Metric
- removed TP_3.3V1, TP_Vbias1: TestPoint, TestPoint:TestPoint_Pad_D1.0mm
- added CS15: 100n, Capacitor_SMD:C_0603_1608Metric, F.Cu at (84.6, 99.2)
- added CS31: 10u, Capacitor_SMD:C_0603_1608Metric, F.Cu at (98.4, 58.1)
- added CS32: 100n, Capacitor_SMD:C_0603_1608Metric, F.Cu at (100.9, 57.6)
- added CS33: 10n, Capacitor_SMD:C_0603_1608Metric, F.Cu at (100.1, 64.1)
- added CS34: 10u, Capacitor_SMD:C_0603_1608Metric, F.Cu at (98.4, 61.1)
- added IC5: TPS7A9101DSKR, TPS7A9101DSKR:SON50P250X250X80-11N-D, F.Cu at (100.9, 60.6)
- added R32: 1.15k, Resistor_SMD:R_0603_1608Metric, F.Cu at (101.9, 64.1)
- added R33: 3.57k, Resistor_SMD:R_0603_1608Metric, F.Cu at (98.4, 64.1)
- added Rf_Opamp1: 0R, Resistor_SMD:R_0603_1608Metric, F.Cu at (88.9, 95.8)
- added TP_3.3V2: TestPoint, TestPoint:TestPoint_Pad_D1.5mm, B.Cu at (95.7, 61.9)
- added TP_CS1: TestPoint, TestPoint:TestPoint_Pad_D1.0mm, F.Cu at (90.7, 67.0)
- added TP_GND3: TestPoint, TestPoint:TestPoint_Pad_D1.0mm, F.Cu at (96.9, 66.3)
- added TP_MISO1: TestPoint, TestPoint:TestPoint_Pad_D1.0mm, F.Cu at (92.8, 69.0)
- added TP_MOSI1: TestPoint, TestPoint:TestPoint_Pad_D1.0mm, F.Cu at (90.7, 69.0)
- added TP_SCLK1: TestPoint, TestPoint:TestPoint_Pad_D1.0mm, F.Cu at (92.8, 67.0)
- added TP_SHIELD1: TestPoint, TestPoint:TestPoint_Pad_D1.5mm, B.Cu at (109.1, 89.4)
- added TP_VBIAS1: TestPoint, TestPoint:TestPoint_Pad_D1.5mm, B.Cu at (90.6, 100.1)
- ADC_Daisy1, ADC_TESTN1, ADC_TESTP1, TP_GND1, TP_GND2, TP_OP_N1, TP_OP_OUT1, TP_OP_P1, TP_REFp1: footprint TestPoint:TestPoint_Pad_D1.0mm -> TestPoint:TestPoint_Pad_D1.5mm
- CF1, CF2, CF3, CF4, CF5, CF6, CF7, CF8: footprint Capacitor_SMD:C_0603_1608Metric -> Capacitor_SMD:C_0805_2012Metric_Pad1.18x1.45mm_HandSolder
- IC3: value TPS7A8801RTJR -> TLV9051IDBVR; footprint TPS7A8801RTJR:QFN50P400X400X80-21N-D -> TLV9051IDBVR:SOT95P280X145-5N
- RF1, RF2, RF3, RF4, RF5, RF6, RF7, RF8: footprint Resistor_SMD:R_0805_2012Metric -> Resistor_SMD:R_0805_2012Metric_Pad1.20x1.40mm_HandSolder
- moved IC3 39.8 mm to (87.5, 99.2), turned to 180 degrees
- moved J3 9.46 mm to (84.8, 67.6)
- moved J2 9.39 mm to (84.8, 64.4)
- moved S2 8.31 mm to (75.8, 66.5), turned to 90 degrees
- moved TP_GND2 7.76 mm to (101.9, 65.9)
- moved R31 3.11 mm to (80.6, 68.3), turned to 0 degrees
- moved JP_ADC_RefP1 2.74 mm to (87.3, 75.9), turned to 180 degrees
- moved TP_REFp1 2.12 mm to (85.2, 75.9), turned to 90 degrees
- moved CF5 1.96 mm to (94.1, 98.7)
- moved CF3 1.92 mm to (94.2, 74.9)
- moved CS4 1.88 mm to (84.1, 95.8), turned to 90 degrees
- moved RF5 1.76 mm to (94.1, 100.7)
- moved RF3 1.67 mm to (94.2, 72.8)
- moved CS18 1.67 mm to (97.4, 73.2), turned to 90 degrees
- moved CS51 1.67 mm to (99.5, 100.4), turned to -90 degrees
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Connections:
- CS18 pad 1: /ADC/Vref -> /ADC/Vbias
- CS19 pad 1: /ADC/Vref -> /ADC/Vbias
- CS52 pad 1: /ADC/Vref -> /ADC/Vbias
- CS53 pad 1: /ADC/Vref -> /ADC/Vbias
- IC1 pad 1: GND -> /ADC/Vbias
- IC1 pad 11: GND -> /ADC/Vbias
- IC1 pad 13: GND -> /ADC/Vbias
- IC1 pad 15: GND -> /ADC/Vbias
- IC1 pad 3: GND -> /ADC/Vbias
- IC1 pad 35: Net-(IC1-~{PWDN}) -> /ADC/ADC.*PWDN
- IC1 pad 5: GND -> /ADC/Vbias
- IC1 pad 7: GND -> /ADC/Vbias
- IC1 pad 9: GND -> /ADC/Vbias
- IC3 pad 1: /Power_battery/non_reg_in -> /ADC/Vbias
- IC3 pad 2: /Power_battery/non_reg_in -> GND
- IC3 pad 3: GND -> Net-(IC1-OPAMPOUT)
- IC3 pad 4: /Power_battery/non_reg_in -> /ADC/Vbias
- J1 pad 1: /ADC/Vref -> /ADC/Vbias
- J1 pad 2: /ADC/RJ45-Sensitive/B -> /ADC/Charge-Amplifier-Sensitive/Vin_B
- J1 pad 3: /ADC/Vref -> /ADC/Vbias
- J1 pad 4: /ADC/Vref -> /ADC/Vbias
- J1 pad 5: /ADC/RJ45-Sensitive/A -> /ADC/Charge-Amplifier-Sensitive/Vin_A
- J1 pad 6: /ADC/RJ45-Sensitive/C -> /ADC/Charge-Amplifier-Sensitive/Vin_C
- J1 pad 7: /ADC/Vref -> /ADC/Vbias
- J1 pad 8: /ADC/RJ45-Sensitive/D -> /ADC/Charge-Amplifier-Sensitive/Vin_D
- J3 pad 1: Net-(IC1-~{PWDN}) -> /ADC/ADC.*PWDN
- J5 pad 1: /ADC/Vref -> /ADC/Vbias
- J5 pad 2: /ADC/RJ45-Coarse/B -> /ADC/Charge-Amplifier-Coarse/Vin_B
- J5 pad 3: /ADC/Vref -> /ADC/Vbias
- J5 pad 4: /ADC/Vref -> /ADC/Vbias
- J5 pad 5: /ADC/RJ45-Coarse/A -> /ADC/Charge-Amplifier-Coarse/Vin_A
- J5 pad 6: /ADC/RJ45-Coarse/C -> /ADC/Charge-Amplifier-Coarse/Vin_C
- J5 pad 7: /ADC/Vref -> /ADC/Vbias
- J5 pad 8: /ADC/RJ45-Coarse/D -> /ADC/Charge-Amplifier-Coarse/Vin_D
- R31 pad 1: Net-(IC1-~{PWDN}) -> /ADC/ADC.*PWDN
- U1 pad 10: /ADC/Vref -> /ADC/Vbias
- U1 pad 12: /ADC/Vref -> /ADC/Vbias
- U1 pad 3: /ADC/Vref -> /ADC/Vbias
- U1 pad 5: /ADC/Vref -> /ADC/Vbias
- U2 pad 10: unconnected-(U2-IO6-Pad10) -> /ADC/ADC.*PWDN
- U2 pad 8: /ADC/Vref -> unconnected-(U2-IO4-Pad8)
- U4 pad 10: /ADC/Vref -> /ADC/Vbias
- U4 pad 12: /ADC/Vref -> /ADC/Vbias
- U4 pad 3: /ADC/Vref -> /ADC/Vbias
- U4 pad 5: /ADC/Vref -> /ADC/Vbias
Routing:
- net /ADC/Vbias: track 0.00 -> 136.7 mm, vias 0 -> 6
- net /ADC/Vref: track 121.2 -> 0.00 mm, vias 7 -> 0
- net /Power_battery/non_reg_in: track 54.3 -> 100.0 mm, vias 2 -> 5
- net /ADC/ADC.*PWDN: track 0.00 -> 38.9 mm, vias 0 -> 2
- net Net-(IC1-~{PWDN}): track 28.3 -> 0.00 mm, vias 1 -> 0
- net /ADC/RJ45-Sensitive/B: track 25.9 -> 0.00 mm
- net /ADC/Charge-Amplifier-Coarse/Vin_B: track 9.79 -> 34.5 mm, vias 2 -> 1
- net /ADC/Charge-Amplifier-Sensitive/Vin_B: track 10.6 -> 35.0 mm, vias 2 -> 1
- net /ADC/RJ45-Coarse/A: track 23.1 -> 0.00 mm
- net /ADC/Charge-Amplifier-Coarse/Vin_A: track 10.7 -> 31.3 mm, vias 2 -> 1
- net /ADC/Charge-Amplifier-Sensitive/Vin_A: track 10.8 -> 31.1 mm, vias 2 -> 1
- net /ADC/RJ45-Sensitive/A: track 19.2 -> 0.00 mm
- net /ADC/AVDD: track 137.1 -> 118.4 mm, vias 7 -> 5
- net /ADC/RJ45-Coarse/B: track 15.5 -> 0.00 mm, vias 1 -> 0
- net /ADC/Charge-Amplifier-Sensitive/Vin_D: track 10.5 -> 25.7 mm, vias 2 -> 1
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Other:
- board text added: "CH1/D"
- board text added: "CH2/C"
- board text added: "CH3/B"
- board text added: "CH4/A"
- board text added: "CH5/D"
- board text added: "CH6/C"
- board text added: "CH7/B"
- board text added: "CH8/A"
- board text added: "COARSE"
- board text added: "CS CLK"
- board text added: "CS MISO CLK MOSI"
- board text added: "IO2 GND"
- board text added: "IO3 GND"
- board text added: "MOSI MISO"
- board text added: "PINOUT RJ45 (T-568B) 5(4) A/blue 2(1) B/orange 6(3) C/green 8(7) D/brown full(striped) Pin(Vbias)"
- board text added: "SENSITIVE"
- board text added: "Schlaubi-Schlumpf v1.1 (Multi-Ferro-DAQ) Mark Suppelt"
- board text added: "striped (1,3,4,7) Vbias full (2,5,6,8) signal"
- board text removed: "*PWDN"
- board text removed: "*RESET"
- board text removed: "GPIO2"
- board text removed: "GPIO3"
- board text removed: "PINOUT RJ45 (T-568B) 1+2 orange/B 3+6 green/C 4+5 blue/A 7+8 brown/D (striped + full) (Vref+Pin)"
- board text removed: "Schlaubi-Schlumpf v1.0 (Multi-Ferro-DAQ) Mark Suppelt"
- board text removed: "striped (1,3,4,7) on Vref"

Commit message: newest order 17.09
Parts:
- removed R31: 10k, Resistor_SMD:R_0603_1608Metric
- removed SPIEXT1: Conn_01x04_Pin, Connector_PinHeader_1.27mm:PinHeader_1x04_P1.27mm_Vertical
- added CS_External1: TestPoint, TestPoint:TestPoint_THTPad_D1.0mm_Drill0.5mm, F.Cu at (87.0, 45.4)
- added TP_DRDY1: TestPoint, TestPoint:TestPoint_Pad_D1.0mm, B.Cu at (78.0, 74.8)
- ADC_Daisy1, ADC_TESTN1, ADC_TESTP1, TP_3.3V2, TP_GND1, TP_GND2, TP_OP_N1, TP_OP_OUT1, TP_OP_P1, TP_REFp1, TP_SHIELD1, TP_VBIAS1: footprint TestPoint:TestPoint_Pad_D1.5mm -> TestPoint:TestPoint_Pad_D1.0mm
- CF1, CF2, CF3, CF4: value 330p -> 330n
- R27: value 0R -> 27R
- RF1, RF2, RF3, RF4: value 2G -> 15k
- moved G*** 2.68 mm to (96.9, 80.2)
- moved ADC_TESTP1 0.89 mm to (90.7, 81.5)
- moved TP_CS1 0.10 mm to (90.7, 66.9)
- moved TP_SCLK1 0.10 mm to (92.8, 66.9)
Routing:
- net /ADC/ADC.*PWDN: track 38.9 -> 32.1 mm
- net /ESP32/IMU.CS: track 9.01 -> 4.85 mm
- net /ESP32/IMU.SDO/MISO: track 6.76 -> 5.13 mm, vias 1 -> 0
- net /ADC/DVDD: track 136.8 -> 135.3 mm
- net GND: track 101.2 -> 100.2 mm
- net /ESP32/IMU.SDA/MOSI: track 9.22 -> 8.35 mm, vias 0 -> 2
- net /ESP32/IMU.SCL/SCLK: track 11.0 -> 11.9 mm, vias 1 -> 3
- net /ESP32/IMU.Interrupt: track 9.18 -> 9.99 mm, vias 2 -> 0
- net /ADC/ADC.*DRDY: track 42.9 -> 43.3 mm, vias 0 -> 1
- net Shield: vias 41 -> 83
Other:
- board text added: "2 B"
- board text added: "5 A"
- board text added: "6 C"
- board text added: "8 D"
- board text added: "IN1"
- board text added: "IN8"
- board text added: "PINOUT RJ45(T-568B) Pin(V_Bias) - Channel 5(4) - A/blue 2(1) - B/orange 6(3) - C/green 8(7) - D/brown Pin = full color (Vbias) = striped"
- board text added: "Schlaubi-Schlumpf v1.2 (Multi-Ferro-DAQ) Mark Suppelt"
- board text removed: "2"
- board text removed: "5"
- board text removed: "6"
- board text removed: "8"
- board text removed: "CS MISO CLK MOSI"
- board text removed: "MOSI SCLK MISO CS"
- board text removed: "PINOUT RJ45 (T-568B) 5(4) A/blue 2(1) B/orange 6(3) C/green 8(7) D/brown full(striped) Pin(Vbias)"
- board text removed: "SDA SCL SDO CS"
- board text removed: "Schlaubi-Schlumpf v1.1 (Multi-Ferro-DAQ) Mark Suppelt"

Commit message: corrected cap/resistor
Parts:
- CF1, CF2, CF3, CF4, CF5, CF6, CF7, CF8: value 330n -> 680p
- RF1, RF2, RF3, RF4, RF5, RF6, RF7, RF8: value 15k -> 1G
Changed lines of the file:
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@@
 			)
 		)
-		(property "Value" "15k"
+		(property "Value" "1G"
 			(at 0 1.65 0)
 			(layer "F.Fab")
@@
 			)
 		)
-		(property "LCSC" "C17475"
+		(property "LCSC" "C2484710"
 			(at 0 0 0)
 			(layer "F.SilkS")
@@
 			)
 		)
-		(property "Value" "330n"
+		(property "Value" "680p"
 			(at 0 1.68 0)
 			(layer "F.Fab")
@@
 			)
 		)
-		(property "LCSC" "C1740"
+		(property "LCSC" "C1754"
 			(at 0 0 0)
 			(layer "F.SilkS")
@@
 			)
 		)
-		(property "Value" "330n"
+		(property "Value" "680p"
 			(at 0 1.68 0)
 			(layer "F.Fab")
@@
 			)
 		)
-		(property "LCSC" "C1740"
+		(property "LCSC" "C1754"
 			(at 0 0 0)
 			(layer "F.SilkS")
@@
 			)
 		)
-		(property "Value" "15k"
+		(property "Value" "1G"
 			(at 0 1.65 0)
 			(layer "F.Fab")
@@
 			)
 		)
-		(property "LCSC" "C17475"
+		(property "LCSC" "C2484710"
 			(at 0 0 0)
 			(layer "F.SilkS")
@@
 			)
 		)
-		(property "Value" "15k"
+		(property "Value" "1G"
 			(at 0 1.65 0)
 			(layer "F.Fab")
@@
 			)
 		)
-		(property "LCSC" "C17475"
+		(property "LCSC" "C2484710"
 			(at 0 0 0)
 			(layer "F.SilkS")
@@
 			)
 		)
-		(property "Value" "330n"
+		(property "Value" "680p"
 			(at 0 1.68 0)
 			(layer "F.Fab")
@@
 			)
 		)
-		(property "LCSC" "C1740"
+		(property "LCSC" "C1754"
 			(at 0 0 0)
 			(layer "F.SilkS")
@@
 		(tags "capacitor")
 		(property "Reference" "CS17"
-			(at -1 0.99 0)
+			(at -1 0.79 0)
 			(unlocked yes)
 			(layer "F.SilkS")
@@
 			)
 		)
-		(property "Value" "15k"
+		(property "Value" "1G"
 			(at 0 1.65 0)
 			(layer "F.Fab")
@@
 			)
 		)
-		(property "LCSC" "C17475"
+		(property "LCSC" "C2484710"
 			(at 0 0 0)
 			(layer "F.SilkS")
@@
 		(sheetname "/ESP32/")
 		(sheetfile "ESP32.kicad_sch")
-		(attr exclude_from_pos_files exclude_from_bom)
+		(attr exclude_from_pos_files)
 		(fp_circle
 			(center 0 0)
@@
 			)
 		)
-		(property "Value" "15k"
+		(property "Value" "1G"
 			(at 0 1.65 0)
 			(layer "F.Fab")
@@
 			)
 		)
-		(property "LCSC" "C17475"
+		(property "LCSC" "C2484710"
 			(at 0 0 0)
 			(layer "F.SilkS")
@@
 		(tags "resistor handsolder")
 		(property "Reference" "RF2"
-			(at -1.9 0 90)
+			(at 1.9 0 270)
 			(unlocked yes)
 			(layer "F.SilkS")
@@
 			)
 		)
-		(property "Value" "15k"
+		(property "Value" "1G"
 			(at 0 1.65 0)
 			(layer "F.Fab")
@@
 			)
 		)
-		(property "LCSC" "C17475"
+		(property "LCSC" "C2484710"
 			(at 0 0 0)
 			(layer "F.SilkS")
@@
 		(tags "capacitor handsolder")
 		(property "Reference" "CF2"
-			(at -2 0 90)
+			(at 1.9 0 270)
 			(unlocked yes)
 			(layer "F.SilkS")
@@
 			)
 		)
-		(property "Value" "330n"
+		(property "Value" "680p"
 			(at 0 1.68 0)
 			(layer "F.Fab")
@@
 			)
 		)
-		(property "LCSC" "C1740"
+		(property "LCSC" "C1754"
 			(at 0 0 0)
 			(layer "F.SilkS")
@@
 		(sheetname "/ESP32/")
 		(sheetfile "ESP32.kicad_sch")
-		(attr exclude_from_pos_files exclude_from_bom)
+		(attr exclude_from_pos_files)
 		(fp_circle
 			(center 0 0)
@@
 		(tags "resistor handsolder")
 		(property "Reference" "RF8"
-			(at -2 0 90)
+			(at 1.9 0 270)
 			(unlocked yes)
 			(layer "F.SilkS")
@@
 			)
 		)
-		(property "Value" "15k"
+		(property "Value" "1G"
 			(at 0 1.65 0)
 			(layer "F.Fab")
@@
 			)
 		)
-		(property "LCSC" "C17475"
+		(property "LCSC" "C2484710"
 			(at 0 0 0)
 			(layer "F.SilkS")
@@
 			)
 		)
-		(property "Value" "15k"
+		(property "Value" "1G"
 			(at 0 1.65 0)
 			(layer "F.Fab")
@@
 			)
 		)
-		(property "LCSC" "C17475"
+		(property "LCSC" "C2484710"
 			(at 0 0 0)
 			(layer "F.SilkS")
@@
 		(tags "capacitor")
 		(property "Reference" "CS28"
-			(at -2.5 -0.15 0)
+			(at -2.2 0.05 0)
 			(unlocked yes)
 			(layer "F.SilkS")
@@
 		(tags "resistor")
 		(property "Reference" "R13"
-			(at 0 -1.1 180)
+			(at -2 0 0)
 			(unlocked yes)
 			(layer "F.SilkS")
@@
 			)
 		)
-		(property "Value" "330n"
+		(property "Value" "680p"
 			(at 0 1.68 0)
 			(layer "F.Fab")
@@
 			)
 		)
-		(property "LCSC" "C1740"
+		(property "LCSC" "C1754"
 			(at 0 0 0)
 			(layer "F.SilkS")
@@
 		(tags "capacitor")
 		(property "Reference" "CS40"
-			(at -1.875 0 90)
+			(at 0.025 -0.8 0)
 			(unlocked yes)
 			(layer "F.SilkS")
@@
 			)
 		)
-		(property "Value" "330n"
+		(property "Value" "680p"
 			(at 0 1.68 0)
 			(layer "F.Fab")
@@
 			)
 		)
-		(property "LCSC" "C1740"
+		(property "LCSC" "C1754"
 			(at 0 0 0)
 			(layer "F.SilkS")
@@
 		(tags "capacitor")
 		(property "Reference" "CS29"
-			(at -2.5 -0.85 0)
+			(at -2.2 0.05 0)
 			(unlocked yes)
 			(layer "F.SilkS")
@@
 		(sheetname "/ESP32/")
 		(sheetfile "ESP32.kicad_sch")
-		(attr exclude_from_pos_files exclude_from_bom)
+		(attr exclude_from_pos_files)
 		(fp_circle
 			(center 0 0)
@@
 		(sheetname "/ESP32/")
 		(sheetfile "ESP32.kicad_sch")
-		(attr exclude_from_pos_files exclude_from_bom)
+		(attr exclude_from_pos_files)
 		(fp_circle
 			(center 0 0)
@@
 		(sheetname "/ESP32/")
 		(sheetfile "ESP32.kicad_sch")
-		(attr exclude_from_pos_files exclude_from_bom)
+		(attr exclude_from_pos_files)
 		(fp_circle
 			(center 0 0)
@@
 			)
 		)
-		(property "Value" "330n"
+		(property "Value" "680p"
 			(at 0 1.68 0)
 			(layer "F.Fab")
@@
 			)
 		)
-		(property "LCSC" "C1740"
+		(property "LCSC" "C1754"
 			(at 0 0 0)
 			(layer "F.SilkS")
@@
 		(tags "capacitor handsolder")
 		(property "Reference" "CF8"
-			(at -2 0 90)
+			(at 1.9 0 270)
 			(unlocked yes)
 			(layer "F.SilkS")
@@
 			)
 		)
-		(property "Value" "330n"
+		(property "Value" "680p"
 			(at 0 1.68 0)
 			(layer "F.Fab")
@@
 			)
 		)
-		(property "LCSC" "C1740"
+		(property "LCSC" "C1754"
 			(at 0 0 0)
 			(layer "F.SilkS")
@@
 		(sheetname "/ESP32/")
 		(sheetfile "ESP32.kicad_sch")
-		(attr exclude_from_pos_files exclude_from_bom)
+		(attr exclude_from_pos_files)
 		(fp_circle
 			(center 0 0)
@@
 		(tags "capacitor")
 		(property "Reference" "CS52"
-			(at 0.9 -1 0)
+			(at 0.9 -0.8 0)
 			(unlocked yes)
 			(layer "F.SilkS")
@@
 		(sheetname "/ADC/")
 		(sheetfile "ADC.kicad_sch")
-		(attr exclude_from_pos_files exclude_from_bom)
+		(attr exclude_from_pos_files)
 		(fp_circle
 			(center 0 0)
@@
 		(sheetname "/ADC/")
 		(sheetfile "ADC.kicad_sch")
-		(attr exclude_from_pos_files exclude_from_bom)
+		(attr exclude_from_pos_files)
 		(fp_circle
 			(center 0 0)
@@
 		(sheetname "/ADC/")
 		(sheetfile "ADC.kicad_sch")
-		(attr exclude_from_pos_files exclude_from_bom)
+		(attr exclude_from_pos_files)
 		(fp_circle
 			(center 0 0)
@@
 		(sheetname "/Power_battery/")
 		(sheetfile "Power.kicad_sch")
-		(attr exclude_from_pos_files exclude_from_bom)
+		(attr exclude_from_pos_files)
 		(fp_circle
 			(center 0 0)
@@
 		(sheetname "/ESP32/")
 		(sheetfile "ESP32.kicad_sch")
-		(attr exclude_from_pos_files exclude_from_bom)
+		(attr exclude_from_pos_files)
 		(fp_circle
 			(center 0 0)
@@
 		(sheetname "/ADC/")
 		(sheetfile "ADC.kicad_sch")
-		(attr exclude_from_pos_files exclude_from_bom)
+		(attr exclude_from_pos_files)
 		(fp_circle
 			(center 0 0)
@@
 		(sheetname "/ADC/")
 		(sheetfile "ADC.kicad_sch")
-		(attr exclude_from_pos_files exclude_from_bom)
+		(attr exclude_from_pos_files)
 		(fp_circle
 			(center 0 0)
@@
 		(sheetname "/ADC/")
 		(sheetfile "ADC.kicad_sch")
-		(attr exclude_from_pos_files exclude_from_bom)
+		(attr exclude_from_pos_files)
 		(fp_circle
 			(center 0 0)
@@
 		(sheetname "/ADC/")
 		(sheetfile "ADC.kicad_sch")
-		(attr exclude_from_pos_files exclude_from_bom)
+		(attr exclude_from_pos_files)
 		(fp_circle
 			(center 0 0)
@@
 		(sheetname "/ADC/")
 		(sheetfile "ADC.kicad_sch")
-		(attr exclude_from_pos_files exclude_from_bom)
+		(attr exclude_from_pos_files)
 		(fp_circle
 			(center 0 0)
@@
 		(sheetname "/ADC/")
 		(sheetfile "ADC.kicad_sch")
-		(attr exclude_from_pos_files exclude_from_bom)
+		(attr exclude_from_pos_files)
 		(fp_circle
 			(center 0 0)
@@
 		(sheetname "/ADC/")
 		(sheetfile "ADC.kicad_sch")
-		(attr exclude_from_pos_files exclude_from_bom)
+		(attr exclude_from_pos_files)
 		(fp_circle
 			(center 0 0)
@@
 		(sheetname "/Power_battery/")
 		(sheetfile "Power.kicad_sch")
-		(attr exclude_from_pos_files exclude_from_bom)
+		(attr exclude_from_pos_files)
 		(fp_circle
 			(center 0 0)
