File: PCB/ESP32.kicad_sch (KiCad schematic)
At the start: 28 parts, among them J2 Conn_01x04_Socket, J3 Conn_01x04_Socket, U2 ESP32-S3-MINI-1-N8

Commit message: Stemma etc.
Parts:
- TP_CS1, TP_DRDY1, TP_MISO1, TP_MOSI1: now left out of the parts list
- renumbered GPIO3 to GPIO1
Changed lines of the file:
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@@
 		(unit 1)
 		(exclude_from_sim no)
-		(in_bom yes)
+		(in_bom no)
 		(on_board yes)
 		(dnp no)
@@
 		(unit 1)
 		(exclude_from_sim no)
-		(in_bom yes)
+		(in_bom no)
 		(on_board yes)
 		(dnp no)
@@
 		(on_board yes)
 		(dnp no)
-		(property "Reference" "GPIO3"
+		(property "Reference" "GPIO1"
 			(at 104.14 78.1051 90)
 			(effects
@@
 			(project "Schlaubi-Schlumpf"
 				(path "/adec948c-82e6-4ad4-8e75-b19e612c0d17/5509f61c-8a57-450f-8279-a49a1ae29ff5"
-					(reference "GPIO3")
+					(reference "GPIO1")
 					(unit 1)
 				)
@@
 		(unit 1)
 		(exclude_from_sim no)
-		(in_bom yes)
+		(in_bom no)
 		(on_board yes)
 		(dnp no)
@@
 		(unit 1)
 		(exclude_from_sim no)
-		(in_bom yes)
-		(on_board yes)
-		(dnp no)
+		(in_bom no)
+		(on_board yes)
+		(dnp no)
