File: PCB/ADC.kicad_sch (KiCad schematic)
At the start: 40 parts, among them IC1 ADS131E08IPAGR, IC3 TLV9051IDBVR

Commit message: Stemma etc.
Parts:
- added CLKSEL1, CLK_EN1: SolderJumper_3_Bridged12, Jumper:SolderJumper-3_P1.3mm_Bridged2Bar12_RoundedPad1.0x1.5mm, symbol Jumper:SolderJumper_3_Bridged12
- added CS20: 1u, Capacitor_SMD:C_0603_1608Metric, symbol Device:C
- added CS22: 100n, Capacitor_SMD:C_0603_1608Metric, symbol Device:C
- added Y1: ASCO, Crystal:Crystal_SMD_3225-4Pin_3.2x2.5mm, symbol Oscillator:ASCO
- ADC_Daisy1, ADC_TESTN1, ADC_TESTP1, TP_ADC_*PWDN1, TP_ADC_*RST1, TP_GND1, TP_OP_N1, TP_OP_OUT1, TP_OP_P1, TP_REFp1, TP_SHIELD1, TP_VBIAS1: now left out of the parts list
Connections:
- net 3.3V: now also CLKSEL1.2 (C), CLKSEL1.3 (B), CLK_EN1.1 (A)
- net GND: now also CLKSEL1.1 (A), CLK_EN1.3 (B), CS20.2, CS22.2, Y1.2 (GND), Y1.3 (OUT)
- new net: CLK_EN1.2 (C), Y1.1 (Tri-State)
- new net: CS20.1, CS22.1, Y1.4 (VDD)
Other:
- note added: "2.048 Mhz OT2EL89CJI-111YLC-2.048M"
- note added: "DVDD - internal CLK GND - external CLK"
- moved on the sheet: TP_ADC_*PWDN1, TP_ADC_*RST1

Commit message: Added Missing Components in Export
Issue was caused by the JLCPCB Plugin which does not export components with a name longer than 7 letters
Parts:
- renumbered Rf_Opamp1 to Rf_Op1
Changed lines of the file:
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@@
 		(on_board yes)
 		(dnp no)
-		(property "Reference" "Rf_Opamp1"
-			(at 124.46 39.624 90)
+		(property "Reference" "Rf_Op1"
+			(at 122.936 52.832 90)
 			(effects
 				(font
 					(size 1.27 1.27)
 				)
-				(hide yes)
 			)
 		)
@@
 			(project "Schlaubi-Schlumpf"
 				(path "/adec948c-82e6-4ad4-8e75-b19e612c0d17/2131c80a-ce05-49b0-92ac-52a13fef390c"
-					(reference "Rf_Opamp1")
+					(reference "Rf_Op1")
 					(unit 1)
 				)
