File: PCB/ADC.kicad_sch (KiCad schematic)
At the start: 45 parts, among them IC1 ADS131E08IPAGR, IC3 TLV9051IDBVR, Y1 ASCO

Commit message: cutout antenna + saved rotation
Parts:
- CS1, CS15, CS3, CS37, CS38: LCSC (none) -> C14663
- CS10, CS12, CS13, CS14, CS4, CS5, CS7, CS8: LCSC (none) -> C15849
- CS11, CS2, CS9: LCSC (none) -> C19702
- CS6: LCSC (none) -> C59461
- D3: LCSC (none) -> C2286
- D4: LCSC (none) -> C2290
- IC1: LCSC (none) -> C190276
- IC3: LCSC (none) -> C1849429
- R1, R2: LCSC (none) -> C25804
- R3, R4, R5: LCSC (none) -> C22775
- Rf_Op1: LCSC (none) -> C21189
