File: PCB/Power.kicad_sch (KiCad schematic)
At the start: 29 parts, among them IC2 TP4056, IC5 TPS7A9101DSKR, IC7 LM2775QDSGRQ1, J4 Conn_01x02_Pin, Q1 DMG2305

Commit message: Stemma etc.
Parts:
- R7: value 4k7 -> 3.57k
- TP_5V1, TP_GND2: now left out of the parts list
Changed lines of the file:
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@@
 		(unit 1)
 		(exclude_from_sim no)
-		(in_bom yes)
+		(in_bom no)
 		(on_board yes)
 		(dnp no)
@@
 			)
 		)
-		(property "Value" "4k7"
+		(property "Value" "3.57k"
 			(at 91.948 105.41 0)
 			(effects
@@
 		(unit 1)
 		(exclude_from_sim no)
-		(in_bom yes)
-		(on_board yes)
-		(dnp no)
+		(in_bom no)
+		(on_board yes)
+		(dnp no)

Commit message: Added Missing Components in Export
Issue was caused by the JLCPCB Plugin which does not export components with a name longer than 7 letters
Parts:
- renumbered CCHARGE1 to CCH1
Changed lines of the file:
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@@
 		(on_board yes)
 		(dnp no)
-		(property "Reference" "CCHARGE1"
+		(property "Reference" "CCH1"
 			(at 114.3 166.37 0)
 			(effects
@@
 			(project "Schlaubi-Schlumpf"
 				(path "/adec948c-82e6-4ad4-8e75-b19e612c0d17/b2b2c764-2d7a-4fe7-b3f5-2bbb716da457"
-					(reference "CCHARGE1")
+					(reference "CCH1")
 					(unit 1)
 				)
