File: PCB/Power.kicad_sch (KiCad schematic)
At the start: 29 parts, among them IC2 TP4056, IC5 TPS7A9101DSKR, IC7 LM2775QDSGRQ1, J4 Conn_01x02_Pin, Q1 DMG2305

Commit message: cutout antenna + saved rotation
Parts:
- C1, C8, C9, CS31, CS34, CS40, CS41: LCSC (none) -> C19702
- CCH1: LCSC (none) -> C15849
- CS32, CS43, CS44: LCSC (none) -> C14663
- CS33: LCSC (none) -> C57112
- D1: LCSC (none) -> C7502695
- D2: LCSC (none) -> C2286
- IC2: LCSC (none) -> C2763448
- IC5: LCSC (none) -> C2878140
- IC7: LCSC (none) -> C2071153
- J4: LCSC (none) -> C594142
- Q1: LCSC (none) -> C2940629
- R17: LCSC (none) -> C25804
- R32: LCSC (none) -> C861724
- R33: LCSC (none) -> C326745
- R6: LCSC (none) -> C21190
- R7: LCSC (none) -> C23162
- S1: LCSC (none) -> C136723
Changed lines of the file:
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@@
+			)
+		)
+		(property "LCSC" "C14663"
+			(at 41.402 150.114 0)
+			(effects
+				(font
+					(size 1.27 1.27)
+				)
+				(hide yes)
 			)
 		)
@@
 			)
 		)
+		(property "LCSC" "C326745"
+			(at 240.03 57.15 0)
+			(effects
+				(font
+					(size 1.27 1.27)
+				)
+				(hide yes)
+			)
+		)
 		(pin "2"
 		)
@@
 			)
 		)
+		(property "LCSC" "C23162"
+			(at 96.7486 105.41 0)
+			(effects
+				(font
+					(size 1.27 1.27)
+				)
+				(hide yes)
+			)
+		)
 		(pin "1"
 		)
@@
 			)
 		)
+		(property "LCSC" "C25804"
+			(at 34.29 46.99 0)
+			(effects
+				(font
+					(size 1.27 1.27)
+				)
+				(hide yes)
+			)
+		)
 		(pin "2"
 		)
@@
 			)
 		)
+		(property "LCSC" "C2286"
+			(at 40.64 102.87 0)
+			(effects
+				(font
+					(size 1.27 1.27)
+				)
+				(hide yes)
+			)
+		)
 		(pin "1"
 		)
@@
 			)
 		)
+		(property "LCSC" "C19702"
+			(at 254.762 64.516 0)
+			(effects
+				(font
+					(size 1.27 1.27)
+				)
+				(hide yes)
+			)
+		)
 		(pin "1"
 		)
@@
 		(property "Description" ""
 			(at 77.47 39.37 0)
+			(effects
+				(font
+					(size 1.27 1.27)
+				)
+				(hide yes)
+			)
+		)
+		(property "LCSC" "C136723"
+			(at 69.8344 34.2797 0)
 			(effects
 				(font
@@
 			)
 		)
+		(property "LCSC" "C2878140"
+			(at 191.77 39.37 0)
+			(effects
+				(font
+					(size 1.27 1.27)
+				)
+				(hide yes)
+			)
+		)
 		(pin "1"
 		)
@@
 			)
 		)
+		(property "LCSC" "C14663"
+			(at 166.624 49.022 0)
+			(effects
+				(font
+					(size 1.27 1.27)
+				)
+				(hide yes)
+			)
+		)
 		(pin "1"
 		)
@@
 			)
 		)
+		(property "LCSC" "C19702"
+			(at 56.642 160.274 0)
+			(effects
+				(font
+					(size 1.27 1.27)
+				)
+				(hide yes)
+			)
+		)
 		(pin "1"
 		)
@@
 		(property "Description" ""
 			(at 52.07 99.06 0)
+			(effects
+				(font
+					(size 1.27 1.27)
+				)
+				(hide yes)
+			)
+		)
+		(property "LCSC" "C21190"
+			(at 48.26 97.5614 0)
 			(effects
 				(font
@@
 			)
 		)
+		(property "LCSC" "C2763448"
+			(at 64.7694 86.3593 0)
+			(effects
+				(font
+					(size 1.27 1.27)
+				)
+				(hide yes)
+			)
+		)
 		(pin "1"
 		)
@@
 			)
 		)
+		(property "LCSC" "C2071153"
+			(at 83.82 144.78 0)
+			(effects
+				(font
+					(size 1.27 1.27)
+				)
+				(hide yes)
+			)
+		)
 		(pin "1"
 		)
@@
 			)
 		)
+		(property "LCSC" "C19702"
+			(at 166.878 42.164 0)
+			(effects
+				(font
+					(size 1.27 1.27)
+				)
+				(hide yes)
+			)
+		)
 		(pin "1"
 		)
@@
 			)
 		)
+		(property "LCSC" "C7502695"
+			(at 48.5775 36.83 0)
+			(effects
+				(font
+					(size 1.27 1.27)
+				)
+				(hide yes)
+			)
+		)
 		(pin "1"
 		)
@@
 		(property "Description" "Generic connector, single row, 01x02, script generated"
 			(at 110.49 93.98 0)
+			(effects
+				(font
+					(size 1.27 1.27)
+				)
+				(hide yes)
+			)
+		)
+		(property "LCSC" "C594142"
+			(at 105.664 83.82 0)
 			(effects
 				(font
@@
 			)
 		)
+		(property "LCSC" "C19702"
+			(at 51.562 150.114 0)
+			(effects
+				(font
+					(size 1.27 1.27)
+				)
+				(hide yes)
+			)
+		)
 		(pin "1"
 		)
@@
 			)
 		)
+		(property "LCSC" "C15849"
+			(at 114.3 166.37 0)
+			(effects
+				(font
+					(size 1.27 1.27)
+				)
+				(hide yes)
+			)
+		)
 		(pin "1"
 		)
@@
 			)
 		)
+		(property "LCSC" "C19702"
+			(at 99.441 94.234 0)
+			(effects
+				(font
+					(size 1.27 1.27)
+				)
+				(hide yes)
+			)
+		)
 		(pin "1"
 		)
@@
 		(property "Description" ""
 			(at 57.15 49.53 0)
+			(effects
+				(font
+					(size 1.27 1.27)
+				)
+				(hide yes)
+			)
+		)
+		(property "LCSC" "C19702"
+			(at 55.626 49.911 0)
 			(effects
 				(font
@@
 			)
 		)
+		(property "LCSC" "C14663"
+			(at 46.482 160.274 0)
+			(effects
+				(font
+					(size 1.27 1.27)
+				)
+				(hide yes)
+			)
+		)
 		(pin "1"
 		)
@@
 			)
 		)
+		(property "LCSC" "C2940629"
+			(at 59.944 33.401 0)
+			(effects
+				(font
+					(size 1.27 1.27)
+				)
+				(hide yes)
+			)
+		)
 		(pin "1"
 		)
@@
 			)
 		)
+		(property "LCSC" "C57112"
+			(at 248.158 56.134 0)
+			(effects
+				(font
+					(size 1.27 1.27)
+				)
+				(hide yes)
+			)
+		)
 		(pin "1"
 		)
@@
 			)
 		)
+		(property "LCSC" "C861724"
+			(at 240.03 72.39 0)
+			(effects
+				(font
+					(size 1.27 1.27)
+				)
+				(hide yes)
+			)
+		)
 		(pin "2"
 		)
@@
 			(effects
 				(font
+					(size 1.27 1.27)
+				)
+				(hide yes)
+			)
+		)
+		(property "LCSC" "C19702"
+			(at 55.626 88.011 0)
+			(effects
+				(font

Commit message: prepare for open hardware release
Parts:
- R7: LCSC C23162 -> C326745
