File: PCB/Schlaubi-Schlumpf.kicad_pcb (KiCad board)
At the start: 4 copper layers, 50 x 65 mm, 150 parts, among them IC1 ADS131E08IPAGR, IC2 TP4056, IC3 TLV9051IDBVR, IC5 TPS7A9101DSKR, IC7 LM2775QDSGRQ1, J1 8P8C_Shielded, J2 Conn_01x04_Socket, J3 Conn_01x04_Socket, J4 Conn_01x02_Pin, J5 8P8C_Shielded, J6 TYPE-C-31-M-12, J7 RFShield_TwoPieces, Q1 DMG2305, U1 AD8608ARUZ-REEL, U2 ESP32-S3-MINI-1-N8, U3 ICM-42670-P, U4 AD8608ARUZ-REEL, U5 WE-TVS-82400102

Commit message: cutout antenna + saved rotation
Parts:
- moved G*** 31.5 mm to (77.3, 74.6)
- moved S2 3.79 mm to (79.3, 68.0), turned to 180 degrees
- moved R13 3.25 mm to (78.3, 64.5), turned to -90 degrees
Routing:
- net /ADC/DVDD: track 148.5 -> 150.6 mm
- net /ESP32/Boot: track 15.4 -> 14.1 mm, vias 2 -> 3
- net GND: track 102.1 -> 103.3 mm, vias 107 -> 105
Other:
- outline, holes or cut-outs redrawn
