File: PCB/Schlaubi-Schlumpf.kicad_sch (KiCad schematic)
At the start: 12 parts, among them J6 TYPE-C-31-M-12, J7 RFShield_TwoPieces, U5 WE-TVS-82400102

Commit message: cutout antenna + saved rotation
Parts:
- CS21: LCSC (none) -> C5360852
- FB1, FB2: LCSC (none) -> C2649308
- H2: LCSC (none) -> C5221843
- J6: LCSC (none) -> C165948
- J7: LCSC (none) -> C5241024
- L1: LCSC (none) -> C2649327
- R19, R20: LCSC (none) -> C23186
- U5: LCSC (none) -> C1975330
Changed lines of the file:
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@@
+			)
+		)
+		(property "LCSC" "C165948"
+			(at 49.53 19.05 0)
+			(effects
+				(font
+					(size 1.27 1.27)
+				)
+				(hide yes)
 			)
 		)
@@
 			)
 		)
+		(property "LCSC" "C5221843"
+			(at 21.59 116.84 0)
+			(effects
+				(font
+					(size 1.27 1.27)
+				)
+				(hide yes)
+			)
+		)
 		(pin "1"
 		)
@@
 			)
 		)
+		(property "LCSC" "C1975330"
+			(at 63.5 63.5 0)
+			(effects
+				(font
+					(size 1.27 1.27)
+				)
+				(hide yes)
+			)
+		)
 		(pin "4"
 		)
@@
 			)
 		)
+		(property "LCSC" "C2649308"
+			(at 92.6592 19.05 0)
+			(effects
+				(font
+					(size 1.27 1.27)
+				)
+				(hide yes)
+			)
+		)
 		(pin "1"
 		)
@@
 		(property "Description" "Resistor"
 			(at 71.12 39.37 0)
+			(effects
+				(font
+					(size 1.27 1.27)
+				)
+				(hide yes)
+			)
+		)
+		(property "LCSC" "C23186"
+			(at 71.12 44.45 0)
 			(effects
 				(font
@@
 			)
 		)
+		(property "LCSC" "C2649327"
+			(at 40.259 64.77 0)
+			(effects
+				(font
+					(size 1.27 1.27)
+				)
+				(hide yes)
+			)
+		)
 		(pin "1"
 		)
@@
 			)
 		)
+		(property "LCSC" "C5241024"
+			(at 139.7 170.8149 0)
+			(effects
+				(font
+					(size 1.27 1.27)
+				)
+				(hide yes)
+			)
+		)
 		(pin "1"
 		)
@@
 		(property "Description" "Resistor"
 			(at 27.94 31.75 0)
+			(effects
+				(font
+					(size 1.27 1.27)
+				)
+				(hide yes)
+			)
+		)
+		(property "LCSC" "C23186"
+			(at 27.94 26.67 0)
 			(effects
 				(font
@@
 			)
 		)
+		(property "LCSC" "C2649308"
+			(at 77.4192 19.05 0)
+			(effects
+				(font
+					(size 1.27 1.27)
+				)
+				(hide yes)
+			)
+		)
 		(pin "1"
 		)
@@
 			(effects
 				(font
+					(size 1.27 1.27)
+				)
+				(hide yes)
+			)
+		)
+		(property "LCSC" "C5360852"
+			(at 85.598 29.464 0)
+			(effects
+				(font
