File: PCB/IMU.kicad_sch (KiCad schematic)
At the start: 9 parts, among them U3 ICM-42670-P

Commit message: cutout antenna + saved rotation
Parts:
- CS46: LCSC (none) -> C14663
- CS47, CS48: LCSC (none) -> C15849
- CS49: LCSC (none) -> C57112
- R15, R16: LCSC (none) -> C25804
- U3: LCSC (none) -> C3288646
Changed lines of the file:
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@@
+			)
+		)
+		(property "LCSC" "C57112"
+			(at 97.028 102.616 0)
+			(effects
+				(font
+					(size 1.27 1.27)
+				)
+				(hide yes)
 			)
 		)
@@
 			)
 		)
+		(property "LCSC" "C25804"
+			(at 203.2 53.594 0)
+			(effects
+				(font
+					(size 1.27 1.27)
+				)
+				(hide yes)
+			)
+		)
 		(pin "2"
 		)
@@
 			)
 		)
+		(property "LCSC" "C25804"
+			(at 208.28 53.594 0)
+			(effects
+				(font
+					(size 1.27 1.27)
+				)
+				(hide yes)
+			)
+		)
 		(pin "2"
 		)
@@
 		(property "Description" "Unpolarized capacitor"
 			(at 81.28 107.95 0)
+			(effects
+				(font
+					(size 1.27 1.27)
+				)
+				(hide yes)
+			)
+		)
+		(property "LCSC" "C15849"
+			(at 84.328 100.076 0)
 			(effects
 				(font
@@
 			)
 		)
+		(property "LCSC" "C3288646"
+			(at 148.59 71.12 0)
+			(effects
+				(font
+					(size 1.27 1.27)
+				)
+				(hide yes)
+			)
+		)
 		(pin "4"
 		)
@@
 		(property "Description" "Unpolarized capacitor"
 			(at 76.2 107.95 0)
+			(effects
+				(font
+					(size 1.27 1.27)
+				)
+				(hide yes)
+			)
+		)
+		(property "LCSC" "C14663"
+			(at 74.168 100.076 0)
 			(effects
 				(font
@@
 			(effects
 				(font
+					(size 1.27 1.27)
+				)
+				(hide yes)
+			)
+		)
+		(property "LCSC" "C15849"
+			(at 89.408 100.076 0)
+			(effects
+				(font
